File: pcb/icyradio.sch (EAGLE design)
At the start: 142 parts, among them J1 TRSJACK, J2 TRSJACK, J3 TRSJACK, U1 ICE40HX8K-CT256, U10 ATSAMS70Q21B-C, U2 EFM32GG11B820F2048GL120, U3 LTC2206, U4 CP2615, U5 DSC1211DE3-C0017, U6 TSCS25A3X1NDGXZAX, U7 MIC5301-1.8YD5, U8 MIC23159, U9 RT820T2, X1 8 MHz, X2 32.768 kHz, X3 DNP

Commit message: Added SPI slave with lots of registers Changed some names and comments Added IRQ logic
Parts:
- added C70, C73, C74, C75, C76, C77: 100nF, Capacitor:CAPACITOR-0603
- added C71, C72: DNP, Capacitor:CAPACITOR-0603
- added R43, R44, R45: 100K Ohms, Resistor:RESISTOR-0603
- added R46, R47, R48, R49: 0 Ohms, Resistor:RESISTOR-0603
- added U11: SI5351C, Silicon Labs:SI5351C
- added U12: DSC1201DE3-50M00000, Microchip:DSC1201DE3-50M00000
- added X4: DNP, Crystal:CRYSTAL_4P
Connections:
- new net !CLK_MNGR_IRQ: R45.1, U11.INTR
- new net !CLK_MNGR_OE: R44.1, U11.!OE
- new net !CLK_MNGR_REFCLK_STDBY: R43.2, U12.!STDBY
- new net DDC_CLK: R49.1
- new net FPGA_GP_CLK1: R48.1
- new net FPGA_GP_CLK2: R47.1
- new net MCU_MAIN_CLK: R46.1
- new net N$60: U11.CLKIN, U12.CLK
- new net N$61: C71.C1, U11.XB, X4.2
- new net N$62: C72.C1, U11.XA, X4.1
- net 3V3: now also C70.C1, C73.C1, C74.C1, C75.C1, C76.C1, C77.C1, R44.2, R45.2, U11.VDD, U11.VDDOA, U11.VDDOB, U11.VDDOC, U11.VDDOD, U12.VDD
- net GND: now also C70.C2, C71.C2, C72.C2, C73.C2, C74.C2, C75.C2, C76.C2, C77.C2, R43.1, U11.GND, U12.GND, X4.GND@0, X4.GND@1
Other:
- note added: "DDC_CLK = 49.152 MHz (for 48 kHz audio sample rate) DDC_CLK = 45.1584 MHz (for 44.1 kHz audio sample rate) FPGA_GP_CLK1 = TBD MHz (general purpose clock) FPGA_GP_CLK2 = TBD MHz (general purpose clock) MCU_MAIN_CLK = TBD MHz (MCU main clock)"

Commit message: Add testbenches Change toolchain flow
Parts:
- added C100, C101, C102, C103, C98, C99: 220pF, Capacitor:CAPACITOR-0603
- added C104, C105, C106, C108, C109, C111, C112, C113, C117, C121, C122, C126, C128, C131, C78, C79, C80, C81, C82, C83, C97: 100nF, Capacitor:CAPACITOR-0603
- added C107, C110: DNP, Capacitor:CAPACITOR-0603
- added C114, C115, C129, C133, C134, C140, C141, C84, C87, C88: 4.7uF, Capacitor:CAPACITOR-0603
- added C116, C119, C124: 470pF, Capacitor:CAPACITOR-0603
- added C118, C123, C125, C127: 100uF, Capacitor:CAPACITOR-1206
- added C120, C130, C85, C86: 10nF, Capacitor:CAPACITOR-0603
- added C132, C135, C136, C138, C139, C89, C90, C91, C92, C95, C96: 1uF, Capacitor:CAPACITOR-0603
- added C137: 10uF, Capacitor:CAPACITOR-0603
- added C93, C94: 22nF, Capacitor:CAPACITOR-0603
- added L10, L11, L12, L7, L8, L9: 1.3uH, Inductor:INDUCTOR-0603
- added L13, L14: (no value), Inductor:INDUCTOR-0603
- added L15, L16, L17, L18: 2.7nH, Inductor:INDUCTOR-0603
- added L19: 2.2uH, Inductor:INDUCTOR-0805
- added L20, L22: 2.2uH, Inductor:INDUCTOR-2.5X2X1.2MM
- added L21: 350nH, Inductor:INDUCTOR-0805
- added L23: 350nH, Inductor:INDUCTOR-0603
- added R50, R51, R62, R63, R66, R69, R71, R72, R73: 100K Ohms, Resistor:RESISTOR-0603
- added R52, R53, R54, R55, R56, R57: 0 Ohms, Resistor:RESISTOR-0603
- added R58, R59: 5.1K Ohms, Resistor:RESISTOR-0603
- added R60: 274K Ohms, Resistor:RESISTOR-0603
- added R61: 294K Ohms, Resistor:RESISTOR-0603
- added R64, R67: 309K Ohms, Resistor:RESISTOR-0603
- added R65: 64.9K Ohms, Resistor:RESISTOR-0603
- added R68: 71.5K Ohms, Resistor:RESISTOR-0603
- added R70: 820 Ohms, Resistor:RESISTOR-0603
- added RFCON2: RFCON-SMA-EDGE, RF Connector:RFCON-SMA-EDGE
- added RFCON3: RFCON-U.FL, RF Connector:RFCON-U.FL
- added U13: DSC1201DE3-50M00000, Microchip:DSC1201DE3-50M00000
- added U14: SI5351C, Silicon Labs:SI5351C
- added U15: MIC23155, Microchip:MIC23155
- added U16: MIC23159, Microchip:MIC23159
- added U17: MIC2019, Microchip:MIC2019
- added U18: ADP150UJZ-1.8, Analog Devices:ADP150UJZ-1.8
- added U19: ADP150UJZ-3.3, Analog Devices:ADP150UJZ-3.3
- added U20, U21: MIC94305, Microchip:MIC94305
- C10: value 4.7uF -> 2.2uF
- C11, C56: value 10nF -> 100nF
- C12: value 1uF -> 12pF
- C13: value 100nF -> 12pF
- C14: value 330pF -> 12pF
- C15: value 6.8nF -> 1uF
- C17, C18: value DNP -> 100nF
- C19: value 100nF -> 6.8nF
- C2, C3, C4: value 12pF -> 100nF
- C21: value 100nF -> 2.2uF
- C24, C28: value 100nF -> 330pF
- C29: value 2.2uF -> 10nF
- C30, C42, C55, C57: value 1uF -> 100nF
- C33: value 100nF -> 1uF
- C37, C38, C39, C58: value 4.7uF -> 100nF
- C41: value 10nF -> 100pF
- C43, C44, C51, C52: value 220pF -> 200pF
- C45, C46: value 1uF -> 200pF
- C47, C50: value 1uF -> 620pF
- C48, C49: value 220pF -> 620pF
- C53, C54: value 22nF -> 200pF
- C6: value 2.2uF -> 100nF
- C60: value 100uF -> 100nF; device Capacitor:CAPACITOR-1206 -> Capacitor:CAPACITOR-0603; VOLTAGE 6.3V -> (none)
- C61: value 470pF -> 10nF
- C62: value 470pF -> 100nF
- C63: value 4.7uF -> 10pF
- C65, C67: value 100nF -> 10pF
- C66: value 100uF -> 100nF; device Capacitor:CAPACITOR-1206 -> Capacitor:CAPACITOR-0603
- C68: value 100uF -> 0.4pF; device Capacitor:CAPACITOR-1206 -> Capacitor:CAPACITOR-0603
- C69, C75, C76: value 100nF -> 0.4pF
- C70: value 100nF -> 2.7nF
- C71: value DNP -> 39nF
- C72: value DNP -> 1.3pF
- C73: value 100nF -> 1.3pF
- C74: value 100nF -> 1.2nF
- C8: value 100nF -> DNP
- C9: value 330pF -> DNP
- L1: value 4.7uH -> 150nH; OCLCSC C281111 -> (none); OCMOUSER (none) -> 609-L-14CR15JV4T
- L3: value 150nH -> 8.2nH; OCMOUSER 609-L-14CR15JV4T -> 81-LQW18AN8N2D00D
- L4: value 8.2nH -> 680nH; OCMOUSER 81-LQW18AN8N2D00D -> (none)
- L5: value 2.2uH -> 1.3uH; device Inductor:INDUCTOR-0805 -> Inductor:INDUCTOR-0603; CURRENT 1.2A -> (none); OCLCSC C281115 -> (none)
- L6: value 2.2uH -> 1.3uH; device Inductor:INDUCTOR-2.5X2X1.2MM -> Inductor:INDUCTOR-0603; CURRENT 2.2A -> (none); OCLCSC C375952 -> (none)
- R1: value 25 Ohms -> 100K Ohms
- R11: value 1K Ohms -> 220 Ohms
- R12: value 10K Ohms -> 220 Ohms
- R13: value 5.1K Ohms -> 100K Ohms
- R14: value 5.1K Ohms -> 1.5K Ohms
- R15: value 47K Ohms -> 50 Ohms
- R16: value 24K Ohms -> 50 Ohms
- R17, R18: value 10K Ohms -> 50 Ohms
- R2: value 25 Ohms -> 0 Ohms
- R20: value 4.7K Ohms -> 10K Ohms
- R21, R22: value 600 Ohms -> 100 Ohms
- R23: value 4.7K Ohms -> 100K Ohms
- R24: value 2.21K Ohms -> 4.7K Ohms
- R25: value 2.21K Ohms -> 100 Ohms
- R26: value 4.7K Ohms -> 360 Ohms
- R27: value 600 Ohms -> 680 Ohms
- R28: value 600 Ohms -> 5.1K Ohms
- R29: value 4.7K Ohms -> 5.1K Ohms
- R3: value 25 Ohms -> 1K Ohms
- R30: value 3.57 Ohms -> 10K Ohms
- R31: value 3.57 Ohms -> 24K Ohms
- R32: value 100 Ohms -> 47K Ohms
- R33: value 100 Ohms -> 10K Ohms
- R34: value 309K Ohms -> 100 Ohms
- R35: value 71.5K Ohms -> 2.21K Ohms
- R36, R40: value 100K Ohms -> 4.7K Ohms
- R37: value 274K Ohms -> 4.7K Ohms
- R38: value 294K Ohms -> 10K Ohms
- R39: value 100K Ohms -> 2.21K Ohms
- R41: value 5.1K Ohms -> 4.7K Ohms
- R42: value 5.1K Ohms -> 100 Ohms
- R43, R44: value 100K Ohms -> 600 Ohms
- R45: value 100K Ohms -> 3.57 Ohms
- R46, R47: value 0 Ohms -> 600 Ohms
- R48: value 0 Ohms -> 3.57 Ohms
- R49: value 0 Ohms -> 100K Ohms
- R5: value 220 Ohms -> 25 Ohms
- R6: value 220 Ohms -> 1.8K Ohms
- R7: value DNP -> 25 Ohms
- R8: value 1.8K Ohms -> 25 Ohms
- R9: value 0 Ohms -> DNP
- U1: value ICE40HX8K-CT256 -> EFM32GG11B420F2048GL112; device Lattice:ICE40HX8K-CT256 -> EFM32:EFM32GG11B420F2048GL112
- U10: value ATSAMS70Q21B-C -> ADF4351; device Microchip:ATSAMS70Q21B-C -> Analog Devices:ADF4351
- U11: value SI5351C -> TSCS25A3X1NDGXZAX; device Silicon Labs:SI5351C -> Tempo Semiconductor:TSCS25A3X1NDGXZAX
- U12: value DSC1201DE3-50M00000 -> CP2615; device Microchip:DSC1201DE3-50M00000 -> Silicon Labs:CP2615
- U2: value EFM32GG11B820F2048GL120 -> ATSAMS70Q21B-C; device EFM32:EFM32GG11B820F2048GL120 -> Microchip:ATSAMS70Q21B-C
- U3: value LTC2206 -> ICE40HX8K-CT256; device Analog Devices:LTC2206 -> Lattice:ICE40HX8K-CT256
- U4: value CP2615 -> DSC1211DE3-C0017; device Silicon Labs:CP2615 -> Microchip:DSC1211DE3-C0017
- U5: value DSC1211DE3-C0017 -> LTC2206; device Microchip:DSC1211DE3-C0017 -> Analog Devices:LTC2206
- U6: value TSCS25A3X1NDGXZAX -> RT820T2; device Tempo Semiconductor:TSCS25A3X1NDGXZAX -> Rafael Micro:RT820T2
- U7: value MIC5301-1.8YD5 -> ADL5385; device Microchip:MIC5301-1.8YD5 -> Analog Devices:ADL5385
- U8: value MIC23159 -> AD9117; device Microchip:MIC23159 -> Analog Devices:AD9117
- U9: value RT820T2 -> ADL5545; device Rafael Micro:RT820T2 -> Analog Devices:ADL5545
Connections:
- net TUNER_IF_VAGC renamed RXTUNER_IF_VAGC
- removed net !IFADC_OE: U3.!OE
- removed net 1V2_EN: R40.2, U8.EN@0
- removed net CODEC_1V8: C34.C1, C35.C1, C36.C1, C55.C1, U6.AVDD@0, U6.AVDD@1, U6.CPVDD, U6.DVDD_CORE, U7.OUT
- removed net DDC_CLK: R49.1
- removed net IFADC_CLK: U3.ENC-
- removed net IFADC_D0: U3.D0
- removed net IFADC_D1: U3.D1
- removed net IFADC_D10: U3.D10
- removed net IFADC_D11: U3.D11
- removed net IFADC_D12: U3.D12
- removed net IFADC_D13: U3.D13
- removed net IFADC_D14: U3.D14
- removed net IFADC_D15: U3.D15
- removed net IFADC_D2: U3.D2
- removed net IFADC_D3: U3.D3
- removed net IFADC_D4: U3.D4
- removed net IFADC_D5: U3.D5
- removed net IFADC_D6: U3.D6
- removed net IFADC_D7: U3.D7
- removed net IFADC_D8: U3.D8
- removed net IFADC_D9: U3.D9
- removed net IFADC_DITH: U3.DITH
- removed net IFADC_GAIN: U3.PGA
- removed net IFADC_OF: U3.OF
- removed net IFADC_SHDN: R12.2, U3.SHDN
- removed net IFADC_VCM: C5.C1, C6.C1, R2.2, R3.1, TRF1.CT, U3.VCM
- removed net MCU_DVDD: C10.C1, L1.1, U2.DVDD
- removed net MCU_MAIN_CLK: R46.1
- removed net TUNER_IFN: R5.1, U9.IF_N
- removed net TUNER_IFP: R6.1, U9.IF_P
- removed net TUNER_REFCLK_SEL: U5.FS
- new net !RXADC_OE: U5.!OE
- new net !TXPA_OC: R73.1, U17.!FAULT
- new net 1V8_ANA_CODEC_CLEAN: C138.C1, C80.C1, C82.C1, C83.C1, U11.AVDD@0, U11.AVDD@1, U11.CPVDD, U11.DVDD_CORE, U18.OUT
- new net 3V3_ANA_RX_CLEAN: C10.C1, C141.C1, C16.C1, C18.C1, C2.C1, C20.C1, C22.C1, C4.C1, C6.C1, R3.1, U21.VOUT@0, U21.VOUT@1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
- new net 3V3_ANA_RX_CLEAN_EN: R72.2, U21.EN
- new net 3V3_ANA_TXPLL_CLEAN: C139.C1, C55.C1, C56.C1, C57.C1, C58.C1, C60.C1, L13.1, L14.2, U10.AVDD, U10.SDVDD, U10.VP, U10.VVCO@0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
- new net 3V3_ANA_TX_CLEAN: C140.C1, C34.C1, C36.C1, U20.VOUT@0, U20.VOUT@1, U8.AVDD
- new net 3V3_ANA_TX_CLEAN_EN: R71.2, U20.EN
- new net 3V3_FB1: R64.1, R65.2, U15.FB
- new net 3V6_ANA: C121.C1, C123.C1, C133.C1, C134.C1, C135.C1, C136.C1, L20.2, R64.2, U15.SNS, U18.EN, U18.VIN, U19.EN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
- new net 3V6_ANA_PGOOD: R63.1, U15.PG
- new net 5V0_ANA_TXMIXER_CLEAN: C131.C1, C132.C1, C30.C1, C31.C1, C32.C1, L23.2, U17.VIN, U7.VPS1@0, U7.VPS1@1, U7.VPS2, U7.VPS3@0, U7.VPS3@1
- new net 5V0_ANA_TXPA_CLEAN: C137.C1, C39.C1, C41.C1, L4.2, U17.VOUT
- new net DSP_MCU_MAIN_CLK: R54.1
- new net FPGA_DDC_CLK: R52.1
- new net FPGA_GP_CLK3: R56.1
- new net N$63: C42.C2, RFCON2.SIGNAL
- new net N$64: C35.C1, U7.VOUT
- new net N$65: L20.1, U15.SW
- new net N$66: C116.C1, U15.SS
- new net N$67: C69.C2, L14.1, L16.1, R25.1, U10.RFOUTA-
- new net N$68: C73.C2, L16.2, L18.1
- new net N$69: C68.C1, L13.2, L15.1, R25.2, U10.RFOUTA+
- new net N$70: C72.C1, L15.2, L17.1
- new net N$71: C75.C1, C77.C1, L17.2
- new net N$72: C76.C2, C78.C1, L18.2
- new net N$73: C44.C2, L6.1, R16.1, U8.IOUTN
- new net N$74: C43.C1, L5.1, R15.2, U8.IOUTP
- new net N$75: C48.C2, L10.1, L6.2
- new net N$76: C47.C1, L5.2, L9.1
- new net N$77: C33.C1, U8.DVDD
- new net N$78: C70.C1, C71.C1, R27.2, U10.CPOUT
- new net N$79: C74.C1, R27.1, U10.VTUNE
- new net N$80: C46.C2, L8.1, R18.1, U8.QOUTN
- new net N$81: C45.C1, L7.1, R17.2, U8.QOUTP
- new net N$82: C50.C2, L12.1, L8.2
- new net N$83: C49.C1, L11.1, L7.2
- new net N$84: C71.C2, R26.2
- new net N$85: C66.C1, C67.C1, U10.TEMP
- new net N$86: C64.C1, C65.C1, U10.VCOM
- new net N$87: C62.C1, C63.C1, U10.VREF
- new net N$88: R24.2, U10.RSET
- new net N$89: C61.C2, U10.REFIN
- new net N$90: C40.C2, C42.C1, L4.1, U9.RFOUT
- new net N$92: C40.C1, R14.1
- new net N$93: C120.C1, D3.2, F1.1, L21.1
- new net N$94: R70.2, U17.ILIMIT
- new net RXADC_CLK: U5.ENC-
- new net RXADC_D0: U5.D0
- new net RXADC_D1: U5.D1
- new net RXADC_D10: U5.D10
- new net RXADC_D11: U5.D11
- new net RXADC_D12: U5.D12
- new net RXADC_D13: U5.D13
- new net RXADC_D14: U5.D14
- new net RXADC_D15: U5.D15
- new net RXADC_D2: U5.D2
- new net RXADC_D3: U5.D3
- new net RXADC_D4: U5.D4
- new net RXADC_D5: U5.D5
- new net RXADC_D6: U5.D6
- new net RXADC_D7: U5.D7
- new net RXADC_D8: U5.D8
- new net RXADC_D9: U5.D9
- new net RXADC_DITH: U5.DITH
- new net RXADC_GAIN: U5.PGA
- new net RXADC_OF: U5.OF
- new net RXADC_SHDN: R1.1, U5.SHDN
- new net RXADC_VCM: C21.C1, C23.C1, R7.1, R8.2, TRF1.CT, U5.VCM
- new net RXTUNER_IFN: R12.1, U6.IF_N
- new net RXTUNER_IFP: R11.1, U6.IF_P
- new net RXTUNER_REFCLK_SEL: U4.FS
- new net SMC_MCU_MAIN_CLK: R57.1
- new net TXDAC_AUXI: R19.2, U8.FSADJI/AUXI
- new net TXDAC_AUXQ: R20.2, U8.FSADJQ/AUXQ
- new net TXDAC_D0: U8.DB0
- new net TXDAC_D1: U8.DB1
- new net TXDAC_D10: U8.DB10
- new net TXDAC_D11: U8.DB11
- new net TXDAC_D12: U8.DB12
- new net TXDAC_D13: U8.DB13
- new net TXDAC_D2: U8.DB2
- new net TXDAC_D3: U8.DB3
- new net TXDAC_D4: U8.DB4
- new net TXDAC_D5: U8.DB5
- new net TXDAC_D6: U8.DB6
- new net TXDAC_D7: U8.DB7
- new net TXDAC_D8: U8.DB8
- new net TXDAC_D9: U8.DB9
- new net TXPA_BIAS_EN: R69.2, U17.EN
- new net TXPLL_EN: R23.2, U10.CE
- new net TX_MIXER_EN: R13.2, U7.ENBL
- new net TX_MIXER_IBBN: C52.C2, L10.2, R19.1, R21.1, U7.IBBN
- new net TX_MIXER_IBBP: C51.C1, L9.2, R21.2, U7.IBBP
- new net TX_MIXER_LON: C78.C2, U7.LOIN
- new net TX_MIXER_LOP: C77.C2, U7.LOIP
- new net TX_MIXER_QBBN: C54.C2, L12.2, R20.1, R22.1, U7.QBBN
- new net TX_MIXER_QBBP: C53.C1, L11.2, R22.2, U7.QBBP
- net !CLK_MNGR_IRQ: now also R51.1, U14.INTR; no longer R45.1, U11.INTR
- net !CLK_MNGR_OE: now also R50.1, U14.!OE; no longer R44.1, U11.!OE
- net !CLK_MNGR_REFCLK_STDBY: now also R49.2, U13.!STDBY; no longer R43.2, U12.!STDBY
- net !CODEC_RST: now also R30.1, U11.!RST; no longer R19.1, U6.!RST
- net !I2S_BRG_CFG: now also R33.1, U12.!CFGMODE; no longer R18.1, U4.!CFGMODE
- net !I2S_BRG_RST: now also R38.1, U12.!RST; no longer R17.1, U4.!RST
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Other:
- note added: "FPGA_DDC_CLK = 49.152 MHz (for 48 kHz audio sample rate) FPGA_DDC_CLK = 45.1584 MHz (for 44.1 kHz audio sample rate) FPGA_GP_CLK1 = TBD MHz (general purpose clock) FPGA_GP_CLK2 = TBD MHz (general purpose clock) MCU_MAIN_CLK = TBD MHz (MCU main clock)"
- note removed: "DDC_CLK = 49.152 MHz (for 48 kHz audio sample rate) DDC_CLK = 45.1584 MHz (for 44.1 kHz audio sample rate) FPGA_GP_CLK1 = TBD MHz (general purpose clock) FPGA_GP_CLK2 = TBD MHz (general purpose clock) MCU_MAIN_CLK = TBD MHz (MCU main clock)"

Commit message: Huge PCB layout progress
Parts:
- removed C1, C132, C135, C136, C138, C139, C15, C33, C89, C90, C91, C92, C95, C96: 1uF, Capacitor:CAPACITOR-0603
- removed C10, C21: 2.2uF, Capacitor:CAPACITOR-0603
- removed C100, C98, C99: 220pF, Capacitor:CAPACITOR-0603
- removed C11, C112, C113, C117, C121, C122, C126, C128, C131, C16, C17, C18, C2, C20, C22, C23, C25, C26, C27, C3, C30, C31, C32, C34, C35, C36, C37, C38, C39, C4, C42, C5, C55, C56, C57, C58, C59, C6, C60, C62, C64, C66, C7, C77, C78, C79, C80, C81, C82, C83, C97: 100nF, Capacitor:CAPACITOR-0603
- removed C114, C115, C129, C133, C134, C140, C141, C84, C87, C88: 4.7uF, Capacitor:CAPACITOR-0603
- removed C116, C119, C124: 470pF, Capacitor:CAPACITOR-0603
- removed C118, C123, C125, C127: 100uF, Capacitor:CAPACITOR-1206
- removed C12, C13, C14: 12pF, Capacitor:CAPACITOR-0603
- removed C120, C130, C29, C40, C61, C85, C86: 10nF, Capacitor:CAPACITOR-0603
- removed C137: 10uF, Capacitor:CAPACITOR-0603
- removed C19: 6.8nF, Capacitor:CAPACITOR-0603
- removed C24, C28: 330pF, Capacitor:CAPACITOR-0603
- removed C41: 100pF, Capacitor:CAPACITOR-0603
- removed C43, C44, C45, C46, C51, C52, C53, C54: 200pF, Capacitor:CAPACITOR-0603
- removed C47, C48, C49, C50: 620pF, Capacitor:CAPACITOR-0603
- removed C63, C65, C67: 10pF, Capacitor:CAPACITOR-0603
- removed C68, C69, C75, C76: 0.4pF, Capacitor:CAPACITOR-0603
- removed C70: 2.7nF, Capacitor:CAPACITOR-0603
- removed C71: 39nF, Capacitor:CAPACITOR-0603
- removed C72, C73: 1.3pF, Capacitor:CAPACITOR-0603
- removed C74: 1.2nF, Capacitor:CAPACITOR-0603
- removed C8, C9: DNP, Capacitor:CAPACITOR-0603
- removed C93, C94: 22nF, Capacitor:CAPACITOR-0603
- removed D1: BAV99, Generic Diode:BAV99
- removed D2, D3: SP0503BAHT, TVS:SP0503BAHT
- removed F1: (no value), PTC Fuses:PTC1206
- removed J1, J2, J3: TRSJACK, DC Jack:TRSJACK
- removed L1, L2: 150nH, Inductor:INDUCTOR-0603
- removed L10, L11, L12, L5, L6, L7, L8, L9: 1.3uH, Inductor:INDUCTOR-0603
- removed L13, L14: (no value), Inductor:INDUCTOR-0603
- removed L15, L16, L17, L18: 2.7nH, Inductor:INDUCTOR-0603
- removed L19: 2.2uH, Inductor:INDUCTOR-0805
- removed L20, L22: 2.2uH, Inductor:INDUCTOR-2.5X2X1.2MM
- removed L21: 350nH, Inductor:INDUCTOR-0805
- removed L23: 350nH, Inductor:INDUCTOR-0603
- removed L3: 8.2nH, Inductor:INDUCTOR-0603
- removed L4: 680nH, Inductor:INDUCTOR-0603
- removed R10, R19, R20, R30, R33, R38: 10K Ohms, Resistor:RESISTOR-0603
- removed R11, R12: 220 Ohms, Resistor:RESISTOR-0603
- removed R13, R23, R49, R50, R51, R62, R63, R66, R69, R71, R72, R73: 100K Ohms, Resistor:RESISTOR-0603
- removed R14: 1.5K Ohms, Resistor:RESISTOR-0603
- removed R15, R16, R17, R18: 50 Ohms, Resistor:RESISTOR-0603
- removed R21, R22, R25, R34, R42: 100 Ohms, Resistor:RESISTOR-0603
- removed R24, R36, R37, R40, R41: 4.7K Ohms, Resistor:RESISTOR-0603
- removed R26: 360 Ohms, Resistor:RESISTOR-0603
- removed R27: 680 Ohms, Resistor:RESISTOR-0603
- removed R28, R29, R58, R59: 5.1K Ohms, Resistor:RESISTOR-0603
- removed R31: 24K Ohms, Resistor:RESISTOR-0603
- removed R32: 47K Ohms, Resistor:RESISTOR-0603
- removed R35, R39: 2.21K Ohms, Resistor:RESISTOR-0603
- removed R43, R44, R46, R47: 600 Ohms, Resistor:RESISTOR-0603
- removed R45, R48: 3.57 Ohms, Resistor:RESISTOR-0603
- removed R52, R53, R54, R55, R56, R57: 0 Ohms, Resistor:RESISTOR-0603
- removed R60: 274K Ohms, Resistor:RESISTOR-0603
- removed R61: 294K Ohms, Resistor:RESISTOR-0603
- removed R64, R67: 309K Ohms, Resistor:RESISTOR-0603
- removed R65: 64.9K Ohms, Resistor:RESISTOR-0603
- removed R68: 71.5K Ohms, Resistor:RESISTOR-0603
- removed R7, R8: 25 Ohms, Resistor:RESISTOR-0603
- removed R70: 820 Ohms, Resistor:RESISTOR-0603
- removed R9: DNP, Resistor:RESISTOR-0603
- removed RFCON1, RFCON2: RFCON-SMA-EDGE, RF Connector:RFCON-SMA-EDGE
- removed RFCON3: RFCON-U.FL, RF Connector:RFCON-U.FL
- removed TRF1: ETC1-1T-2TR, Inductor:ETC1-1T-2TR
- removed U1: EFM32GG11B420F2048GL112, EFM32:EFM32GG11B420F2048GL112
- removed U10: ADF4351, Analog Devices:ADF4351
- removed U11: TSCS25A3X1NDGXZAX, Tempo Semiconductor:TSCS25A3X1NDGXZAX
- removed U12: CP2615, Silicon Labs:CP2615
- removed U13: DSC1201DE3-50M00000, Microchip:DSC1201DE3-50M00000
- removed U14: SI5351C, Silicon Labs:SI5351C
- removed U15: MIC23155, Microchip:MIC23155
- removed U16: MIC23159, Microchip:MIC23159
- removed U17: MIC2019, Microchip:MIC2019
- removed U18: ADP150UJZ-1.8, Analog Devices:ADP150UJZ-1.8
- removed U19: ADP150UJZ-3.3, Analog Devices:ADP150UJZ-3.3
- removed U2: ATSAMS70Q21B-C, Microchip:ATSAMS70Q21B-C
- removed U20, U21: MIC94305, Microchip:MIC94305
- removed U3: ICE40HX8K-CT256, Lattice:ICE40HX8K-CT256
- removed U4: DSC1211DE3-C0017, Microchip:DSC1211DE3-C0017
- removed U5: LTC2206, Analog Devices:LTC2206
- removed U6: RT820T2, Rafael Micro:RT820T2
- removed U7: ADL5385, Analog Devices:ADL5385
- removed U8: AD9117, Analog Devices:AD9117
- removed U9: ADL5545, Analog Devices:ADL5545
- removed USB1, USB2: USB-C-16P-SMD-FLAT-SIDE-TYPE-2, USB Connector:USB-C-16P-SMD-FLAT-SIDE-TYPE-2
- removed X1: 8 MHz, Crystal:CRYSTAL2-SMD-5032
- removed X2: 32.768 kHz, Crystal:CRYSTAL2-SMD-3215
- removed X3, X4: DNP, Crystal:CRYSTAL_4P
- added C201, C417, C504, C712, C713, C714, C715, C718, C719, C921, C924, C925, C927, C928: 1uF, Capacitor:CAPACITOR-0603
- added C202, C203, C204, C205, C206, C207, C208, C209, C210, C211, C212, C213, C214, C215, C216, C301, C302, C303, C304, C305, C306, C307, C308, C309, C310, C311, C312, C313, C314, C315, C316, C317, C318, C401, C402, C403, C404, C405, C406, C407, C408, C409, C413, C418, C419, C420, C422, C424, C425, C427, C428, C429, C501, C502, C503, C505, C506, C507, C508, C509, C513, C601, C602, C603, C604, C605, C606, C607, C609, C611, C622, C623, C701, C702, C703, C704, C705, C706, C720, C801, C802, C803, C805, C808, C901, C902, C906, C910, C911, C915, C917, C920: 100nF, Capacitor:CAPACITOR-0603
- added C217, C707, C710, C711, C903, C904, C918, C922, C923, C929, C930: 4.7uF, Capacitor:CAPACITOR-0603
- added C218, C608, C610, C612: 10pF, Capacitor:CAPACITOR-0603
- added C410, C411, C511, C804, C807: DNP, Capacitor:CAPACITOR-0603
- added C412, C423: 2.2uF, Capacitor:CAPACITOR-0603
- added C414, C415, C416: 12pF, Capacitor:CAPACITOR-0603
- added C421: 6.8nF, Capacitor:CAPACITOR-0603
- added C426, C430: 330pF, Capacitor:CAPACITOR-0603
- added C431, C708, C709, C909, C919: 10nF, Capacitor:CAPACITOR-0603
- added C510, C619: 1.2nF, Capacitor:CAPACITOR-0603
- added C512: 68pF, Capacitor:CAPACITOR-0603
- added C514, C515, C516, C517, C522, C523, C524, C525: 200pF, Capacitor:CAPACITOR-0603
- added C518, C519, C520, C521: 620pF, Capacitor:CAPACITOR-0603
- added C613, C614, C620, C621: 0.4pF, Capacitor:CAPACITOR-0603
- added C615: 39nF, Capacitor:CAPACITOR-0603
- added C616: 2.7nF, Capacitor:CAPACITOR-0603
- added C617, C618: 1.3pF, Capacitor:CAPACITOR-0603
- added C716, C717: 22nF, Capacitor:CAPACITOR-0603
- added C721, C722, C723, C724, C725, C726: 220pF, Capacitor:CAPACITOR-0603
- added C905, C908, C913: 470pF, Capacitor:CAPACITOR-0603
- added C907, C912, C914, C916: 100uF, Capacitor:CAPACITOR-1206
- added C926: 10uF, Capacitor:CAPACITOR-0603
- added D401: BAV99, Generic Diode:BAV99
- added D701, D901: SP0503BAHT, TVS:SP0503BAHT
- added F901: (no value), PTC Fuses:PTC1206
- added J701, J702, J703: TRSJACK, DC Jack:TRSJACK
- added L201, L202: 470 Ohms, Inductor:INDUCTOR-0603
- added L203: 10uH, Inductor:INDUCTOR-0603
- added L401, L402: 150nH, Inductor:INDUCTOR-0603
- added L403: 8.2nH, Inductor:INDUCTOR-0603
- added L501: 470nH, Inductor:INDUCTOR-0603
- added L502, L503, L504, L505, L506, L507, L508, L509: 1.3uH, Inductor:INDUCTOR-0603
- added L601, L602: 19nH, Inductor:INDUCTOR-0603
- added L603, L604, L605, L606: 2.7nH, Inductor:INDUCTOR-0603
- added L901: 2.2uH, Inductor:INDUCTOR-0805
- added L902, L904: 2.2uH, Inductor:INDUCTOR-2.5X2X1.2MM
- added L903: 350nH, Inductor:INDUCTOR-0805
- added L905: 350nH, Inductor:INDUCTOR-0603
- added R201: 5.62K Ohms, Resistor:RESISTOR-0603
- added R202: 2.2 Ohms, Resistor:RESISTOR-0603
- added R301, R401, R501, R601, R801, R802, R803, R905, R906, R909, R912, R914: 100K Ohms, Resistor:RESISTOR-0603
- added R402, R804, R805, R806, R807, R808, R809: 0 Ohms, Resistor:RESISTOR-0603
- added R403: 1K Ohms, Resistor:RESISTOR-0603
- added R404, R405, R407, R408: 25 Ohms, Resistor:RESISTOR-0603
- added R406: 1.8K Ohms, Resistor:RESISTOR-0603
- added R409, R502, R503, R604: DNP, Resistor:RESISTOR-0603
- added R410, R508, R509, R703, R706, R711: 10K Ohms, Resistor:RESISTOR-0603
- added R411, R412: 220 Ohms, Resistor:RESISTOR-0603
- added R504, R505, R506, R507: 50 Ohms, Resistor:RESISTOR-0603
- added R510, R511, R603, R707, R715: 100 Ohms, Resistor:RESISTOR-0603
- added R602: 5.1K Ohm, Resistor:RESISTOR-0603
- added R605: 360 Ohms, Resistor:RESISTOR-0603
- added R606: 680 Ohms, Resistor:RESISTOR-0603
- added R701, R702, R901, R902: 5.1K Ohms, Resistor:RESISTOR-0603
- added R704: 24K Ohms, Resistor:RESISTOR-0603
- added R705: 47K Ohms, Resistor:RESISTOR-0603
- added R708, R712: 2.21K Ohms, Resistor:RESISTOR-0603
- added R709, R710, R713, R714: 4.7K Ohms, Resistor:RESISTOR-0603
- added R716, R717, R719, R720: 600 Ohms, Resistor:RESISTOR-0603
- added R718, R721: 3.57 Ohms, Resistor:RESISTOR-0603
- added R903: 274K Ohms, Resistor:RESISTOR-0603
- added R904: 294K Ohms, Resistor:RESISTOR-0603
- added R907, R910: 309K Ohms, Resistor:RESISTOR-0603
- added R908: 64.9K Ohms, Resistor:RESISTOR-0603
- added R911: 71.5K Ohms, Resistor:RESISTOR-0603
- added R913: 820 Ohms, Resistor:RESISTOR-0603
- added RFCON401, RFCON501: RFCON-SMA-EDGE, RF Connector:RFCON-SMA-EDGE
- added RFCON502: RFCON-U.FL, RF Connector:RFCON-U.FL
- added TC201: TC2050-IDC, TagConnect:TC2050-IDC
- added TRF401: ETC1-1T-2TR, Inductor:ETC1-1T-2TR
- added U101: EFM32GG11B420F2048GL112, EFM32:EFM32GG11B420F2048GL112
- added U201: ATSAMS70Q21B-C, Microchip:ATSAMS70Q21B-C
- added U301: ICE40HX8K-CT256, Lattice:ICE40HX8K-CT256
- added U401: DSC1211DE3-C0017, Microchip:DSC1211DE3-C0017
- added U402: LTC2206, Analog Devices:LTC2206
- added U403: RT820T2, Rafael Micro:RT820T2
- renumbered TC1 to TC101
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Connections:
- removed net !RST: TC101-10(!RESET!).S
- removed net 1V8_ANA_CODEC_CLEAN: C138.C1, C80.C1, C82.C1, C83.C1, U11.AVDD@0, U11.AVDD@1, U11.CPVDD, U11.DVDD_CORE, U18.OUT
- removed net 3V3_ANA_RX_CLEAN_EN: R72.2, U21.EN
- removed net 3V3_ANA_TX_CLEAN_EN: R71.2, U20.EN
- removed net 3V3_FB1: R64.1, R65.2, U15.FB
- removed net 4V2_FB: R60.1, R61.2, U16.FB@0
- removed net DSP_MCU_MAIN_CLK: R54.1
- removed net MAIN_HFXTAL_N: U1.PB14, X1.1
- removed net MAIN_HFXTAL_P: U1.PB13, X1.2
- removed net MAIN_LFXTAL_N: U1.PB8, X2.2
- removed net MAIN_LFXTAL_P: U1.PB7, X2.1
- removed net MCU_D+: D3.4, USB2.D+
- removed net MCU_D-: D3.3, USB2.D-
- removed net N$20: C15.C1, U6.DET1
- removed net N$21: C24.C1, R6.1, U6.CP
- removed net N$23: C11.C1, U6.VDD_PLL
- removed net N$24: C9.C1, U6.XTALO, X3.2
- removed net N$25: C8.C1, R2.1, U6.XTALI, X3.1
- removed net SMC_MCU_MAIN_CLK: R57.1
- removed net SWCLK: TC101-4(TCK/SWCLK).S
- removed net SWDIO: TC101-2(TMS/SWDIO).S
- removed net SWO: TC101-6(TDO/SWO).S
- removed net TX_MIXER_EN: R13.2, U7.ENBL
- removed net TX_MIXER_IBBN: C52.C2, L10.2, R19.1, R21.1, U7.IBBN
- removed net TX_MIXER_IBBP: C51.C1, L9.2, R21.2, U7.IBBP
- removed net TX_MIXER_LON: C78.C2, U7.LOIN
- removed net TX_MIXER_LOP: C77.C2, U7.LOIP
- removed net TX_MIXER_QBBN: C54.C2, L12.2, R20.1, R22.1, U7.QBBN
- removed net TX_MIXER_QBBP: C53.C1, L11.2, R22.2, U7.QBBP
- new net !DSP_IRQ: U101.PE13, U201.PIOA.PA4
- new net !DSP_RESET: TC201-10(!RESET!).S, U201.PWRCTRL.!RST
- new net !DSP_SPI_SS: U101.PA3, U201.PIOB.PB2
- new net !FPGA_CRESET: R301.2, U101.PB6, U301.PWRCTRL.!CRESET
- new net !FPGA_SPI_CS: U101.PC0, U301.BANK2SPI.!SS!/IOB_108
- new net !FPGA_SRESET: U101.PA5, U301.BANK1.IOR_141_GBIN2
- new net !SMC_RESET: TC101-10(!RESET!).S, U101.!RESET
- new net !TXDAC_CS: R2.1, U101.PE9, U502.!CS!/PWRDN
- new net !TXPLL_MUTE: R4.2, U101.PF8, U602.!PDRF
- new net 1V2_FB: R903.1, R904.2, U902.FB@0
- new net 1V8_CODEC_CLEAN: C702.C1, C704.C1, C705.C1, C927.C1, U701.AVDD@0, U701.AVDD@1, U701.CPVDD, U701.DVDD_CORE, U904.OUT
- new net 3V6_ANA_FB: R907.1, R908.2, U901.FB
- new net CLK_MNGR_I2C_SCL: R6.1, U101.PE5, U802.SCL
- new net CLK_MNGR_I2C_SDA: R5.1, U101.PE4, U802.SDA
- new net DSP_BB_I2S_LRCLK: U201.PIOE.PE0, U301.BANK1.IOR_157
- new net DSP_BB_I2S_SCLK: U201.PIOA.PA20, U301.BANK1.IOR_151
- new net DSP_BB_I2S_SDIN: U201.PIOE.PE2, U301.BANK1.IOR_153
- new net DSP_BB_I2S_SDOUT: U201.PIOE.PE1, U301.BANK1.IOR_161
- new net DSP_D+: D901.4, U201.PWRCTRL.HSDP, USB901.D+
- new net DSP_D-: D901.3, U201.PWRCTRL.HSDM, USB901.D-
- new net DSP_ERASE: U201.PIOB.PB12
- new net DSP_I2S_LRCLK: U201.PIOA.PA15, U301.BANK1.IOR_123
- new net DSP_I2S_MCLK: U201.PIOA.PA0, U301.BANK1.IOR_131
- new net DSP_I2S_SCLK: U201.PIOA.PA1, U301.BANK1.IOR_127
- new net DSP_I2S_SDIN: U201.PIOA.PA16, U301.BANK1.IOR_121
- new net DSP_I2S_SDOUT: U201.PIOA.PA30, U301.BANK1.IOR_133
- new net DSP_MAIN_CLK: R809.1, U201.PIOB.PB9
- new net DSP_SPI_MISO: U101.PA1, U201.PIOD.PD20
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
Commit message: Nothing to do
Parts:
- removed C802, C803, C805, C808, C910, C911, C915, C917, C920: 100nF, Capacitor:CAPACITOR-0603
- removed C804, C807: DNP, Capacitor:CAPACITOR-0603
- removed C908, C913: 470pF, Capacitor:CAPACITOR-0603
- removed C909, C919: 10nF, Capacitor:CAPACITOR-0603
- removed C912, C914, C916: 100uF, Capacitor:CAPACITOR-1206
- removed C918, C922, C923, C929, C930: 4.7uF, Capacitor:CAPACITOR-0603
- removed C921, C924, C925, C927, C928: 1uF, Capacitor:CAPACITOR-0603
- removed C926: 10uF, Capacitor:CAPACITOR-0603
- removed D901: SP0503BAHT, TVS:SP0503BAHT
- removed F901: (no value), PTC Fuses:PTC1206
- removed L901: 2.2uH, Inductor:INDUCTOR-0805
- removed L902, L904: 2.2uH, Inductor:INDUCTOR-2.5X2X1.2MM
- removed L903: 350nH, Inductor:INDUCTOR-0805
- removed L905: 350nH, Inductor:INDUCTOR-0603
- removed R1, R2, R4, R912, R914: 100K Ohms, Resistor:RESISTOR-0603
- removed R3, R806, R807, R808, R809: 0 Ohms, Resistor:RESISTOR-0603
- removed R5, R6: 4.7K Ohms, Resistor:RESISTOR-0603
- removed R910: 309K Ohms, Resistor:RESISTOR-0603
- removed R911: 71.5K Ohms, Resistor:RESISTOR-0603
- removed R913: 820 Ohms, Resistor:RESISTOR-0603
- removed U802: SI5351C, Silicon Labs:SI5351C
- removed U903: MIC2019, Microchip:MIC2019
- removed U904: ADP150UJZ-1.8, Analog Devices:ADP150UJZ-1.8
- removed U905: ADP150UJZ-3.3, Analog Devices:ADP150UJZ-3.3
- removed U906, U907: MIC94305, Microchip:MIC94305
- removed USB901: USB-C-16P-SMD-FLAT-SIDE-TYPE-2, USB Connector:USB-C-16P-SMD-FLAT-SIDE-TYPE-2
- removed X801: DNP, Crystal:CRYSTAL_4P
- added C1001, C1002, C1006, C1010, C1011, C1015, C1017, C1020: 100nF, Capacitor:CAPACITOR-0603
- added C1003, C1004, C1018, C1022, C1023, C1029, C1030: 4.7uF, Capacitor:CAPACITOR-0603
- added C1005, C1008, C1012: 470pF, Capacitor:CAPACITOR-0603
- added C1007, C1013, C1014, C1016: 100uF, Capacitor:CAPACITOR-1206
- added C1009, C1019, C433: 10nF, Capacitor:CAPACITOR-0603
- added C1021, C1024, C1025, C1027, C1028: 1uF, Capacitor:CAPACITOR-0603
- added C1026: 10uF, Capacitor:CAPACITOR-0603
- added C432: 330pF, Capacitor:CAPACITOR-0603
- added C526, C527: 200pF, Capacitor:CAPACITOR-0603
- added D1001: SP0503BAHT, TVS:SP0503BAHT
- added F1001: (no value), PTC Fuses:PTC1206
- added L1001: 2.2uH, Inductor:INDUCTOR-0805
- added L1002, L1004: 2.2uH, Inductor:INDUCTOR-2.5X2X1.2MM
- added L1003: 350nH, Inductor:INDUCTOR-0805
- added L1005: 350nH, Inductor:INDUCTOR-0603
- added Q801, Q802: AO3400, Alpha Omega:AO3400
- added R1001, R1002: 5.1K Ohms, Resistor:RESISTOR-0603
- added R1003: 274K Ohms, Resistor:RESISTOR-0603
- added R1004: 294K Ohms, Resistor:RESISTOR-0603
- added R1005, R1006, R1009, R1012, R1014: 100K Ohms, Resistor:RESISTOR-0603
- added R1007, R1010: 309K Ohms, Resistor:RESISTOR-0603
- added R1008: 64.9K Ohms, Resistor:RESISTOR-0603
- added R101, R102, R103, R104: 4.7K Ohms, Resistor:RESISTOR-0603
- added R1011: 71.5K Ohms, Resistor:RESISTOR-0603
- added R1013: 820 Ohms, Resistor:RESISTOR-0603
- added R105, R203, R414, R512, R513: 10K Ohms, Resistor:RESISTOR-0603
- added R413: DNP, Resistor:RESISTOR-0603
- added R415, R416: 220 Ohms, Resistor:RESISTOR-0603
- added R514, R515: 100 Ohms, Resistor:RESISTOR-0603
- added R607: 680 Ohms, Resistor:RESISTOR-0603
- added SJ1: (no value), Solder Jumper:SJS
- added U1001: MIC23155, Microchip:MIC23155
- added U1002: MIC23159, Microchip:MIC23159
- added U1003: MIC2019, Microchip:MIC2019
- added U1004: ADP150UJZ-1.8, Analog Devices:ADP150UJZ-1.8
- added U1005: ADP150UJZ-3.3, Analog Devices:ADP150UJZ-3.3
- added U1006, U1007: MIC94305, Microchip:MIC94305
- added USB1001: USB-C-16P-SMD-FLAT-SIDE-TYPE-2, USB Connector:USB-C-16P-SMD-FLAT-SIDE-TYPE-2
- added X901: DNP, Crystal:CRYSTAL_4P
- C411, C511: value DNP -> 100nF
- C412: value 2.2uF -> DNP
- C414: value 12pF -> 2.2uF
- C415: value 12pF -> 100nF
- C417: value 1uF -> 12pF
- C419: value 100nF -> 12pF
- C420, C505: value 100nF -> 1uF
- C421: value 6.8nF -> 100nF
- C423: value 2.2uF -> 6.8nF
- C424, C427: value 100nF -> 27pF
- C425: value 100nF -> 2.2uF
- C426, C430: value 330pF -> 100nF
- C428: value 100nF -> 330pF
- C431: value 10nF -> 100nF
- C504: value 1uF -> 100nF
- C510: value 1.2nF -> 100nF
- C512: value 68pF -> 1.2nF
- C513, C906: value 100nF -> DNP
- C514: value 200pF -> 68pF
- C515: value 200pF -> 100nF
- C518, C519: value 620pF -> 200pF
- C522, C523: value 200pF -> 620pF
- C801: value 100nF -> 100uF; device Capacitor:CAPACITOR-0603 -> Capacitor:CAPACITOR-1206
- C903: value 4.7uF -> DNP
- C904: value 4.7uF -> 100nF
- C905: value 470pF -> 100nF
- C907: value 100uF -> 100nF; device Capacitor:CAPACITOR-1206 -> Capacitor:CAPACITOR-0603
- R404, R405: value 25 Ohms -> 220 Ohms
- R406: value 1.8K Ohms -> 25 Ohms
- R408: value 25 Ohms -> 4.7K Ohms
- R409: value DNP -> 1.8K Ohms
- R410: value 10K Ohms -> 4.7K Ohms
- R411, R412: value 220 Ohms -> 25 Ohms
- R502: value DNP -> 0 Ohms
- R503: value DNP -> 100K Ohms
- R504: value 50 Ohms -> 200 Ohms
- R505: value 50 Ohms -> 100K Ohms
- R506, R507: value 50 Ohms -> DNP
- R508, R509: value 10K Ohms -> 50 Ohms
- R510, R511: value 100 Ohms -> 50 Ohms
- R602: value 5.1K Ohm -> 100K Ohms
- R603: value 100 Ohms -> 5.1K Ohm
- R604: value DNP -> 100 Ohms
- R605: value 360 Ohms -> DNP
- R606: value 680 Ohms -> 360 Ohms
- R801: value 100K Ohms -> 22 Ohms
- R802: value 100K Ohms -> 10K Ohms
- R803, R905, R906, R909: value 100K Ohms -> 0 Ohms
- R805: value 0 Ohms -> 100K Ohms
- R901, R902: value 5.1K Ohms -> 100K Ohms
- R903: value 274K Ohms -> 100K Ohms
- R904: value 294K Ohms -> 0 Ohms
- R907: value 309K Ohms -> 0 Ohms
- R908: value 64.9K Ohms -> 0 Ohms
- U801: value DSC1201DE3-50M00000 -> ER-TFT035-6; device Microchip:DSC1201DE3-50M00000 -> BuyDisplay:ER-TFT035-6
- U901: value MIC23155 -> DSC1201DE3-50M00000; device Microchip:MIC23155 -> Microchip:DSC1201DE3-50M00000
- U902: value MIC23159 -> SI5351C; device Microchip:MIC23159 -> Silicon Labs:SI5351C
Connections:
- removed net CLK_MNGR_I2C_SCL: R6.1, U101.PE5, U802.SCL
- removed net CLK_MNGR_I2C_SDA: R5.1, U101.PE4, U802.SDA
- new net !TFT_RESET: U101.PD7, U801.!RESET
- new net !TFT_SPI_CS: R805.1, U101.PA10, U801.!CS
- new net !TFT_TOUCH_IRQ: U101.PD2, U801.X-/!IRQ!
- new net !TFT_TOUCH_RESET: U101.PD3, U801.Y-/!RST!
- new net AUDIO_I2C_SCL: R104.1, U101.PF11, U701.I2C_SCL, U702.I2C_SCL
- new net AUDIO_I2C_SDA: R103.1, U101.PF10, U701.I2C_SDA, U702.I2C_SDA
- new net N$101: Q802.D, R804.1
- new net N$102: Q801.D, R803.1
- new net N$103: Q801.G, Q802.G, R801.1, R802.2
- new net N$104: SJ1.2, TC201-7(RTCK).S
- new net N$20: C424.C1, R405.1, R408.1, U403.SCL
- new net N$21: C427.C1, R404.1, R410.1, U403.SDA
- new net N$23: C507.C1, R504.2, U501.TEMP
- new net N$24: R804.2, U801.LEDK@1
- new net N$25: R803.2, U801.LEDK@0
- new net SYS_I2C_SCL: R102.1, U101.PE5, U801.X+/SCL, U902.SCL
- new net SYS_I2C_SDA: R101.1, U101.PE4, U801.Y+/SDA, U902.SDA
- new net TFT_BL_PWM: R801.2, U101.PD1
- new net TFT_DC: U101.PD4, U801.D/!C!
- new net TFT_SPI_MISO: U101.PA8, U801.SDO
- new net TFT_SPI_MOSI: U101.PA7, U801.SDA
- new net TFT_SPI_SCK: U101.PA9, U801.!WR!/SCL
- new net TXMIXER_TEMP: C510.C1, R504.1, U101.PD6
- net !CLK_MNGR_IRQ: now also R903.1, U101.PE6, U902.INTR; no longer R803.1, U101.PF10, U802.INTR
- net !CLK_MNGR_OE: now also R902.1, U902.!OE; no longer R802.1, U802.!OE
- net !CLK_MNGR_REFCLK_STDBY: now also R901.2, U901.!STDBY; no longer R801.2, U801.!STDBY
- net !CODEC_RST: now also U101.PD0
- net !DSP_RESET: now also R203.1
- net !I2S_BRG_CFG: now also U101.PB12
- net !I2S_BRG_RST: now also U101.PB13
- net !SMC_RESET: now also R105.1
- net !TXDAC_CS: now also R503.1; no longer R2.1
- net !TXPA_OC: now also R1014.1, U1003.!FAULT; no longer R914.1, U903.!FAULT
- net !TXPLL_MUTE: now also R602.2; no longer R4.2
- net 1V2: now also C1006.C1, C1007.C1, L1001.1, R1003.2, U1002.SNS@0; no longer C906.C1, C907.C1, L901.1, R903.2, U902.SNS@0
- net 1V2_FB: now also R1003.1, R1004.2, U1002.FB@0; no longer R903.1, R904.2, U902.FB@0
- net 1V2_PGOOD: now also R1005.1, U1002.PG@0; no longer R905.1, U902.PG@0
- net 1V8_CODEC_CLEAN: now also C1027.C1, U1004.OUT; no longer C927.C1, U904.OUT
- net 3V3: now also C1015.C1, C1016.C1, C1024.C1, C504.C1, C506.C1, C901.C1, C902.C1, C904.C1, C905.C1, C907.C1, L1004.2, R1005.2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; no longer C505.C1, C508.C1, C802.C1, C803.C1, C805.C1, C808.C1, C915.C1, C916.C1, C924.C1, L904.2, R1.2, R2.2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
- net 3V3_ANA_RX_CLEAN: now also C1030.C1, C411.C1, C413.C1, C414.C1, C421.C1, U1007.VOUT@0, U1007.VOUT@1; no longer C412.C1, C420.C1, C422.C1, C424.C1, C930.C1, U907.VOUT@0, U907.VOUT@1
- net 3V3_ANA_TXPLL_CLEAN: now also C1028.C1, U1005.OUT; no longer C928.C1, U905.OUT
- net 3V3_ANA_TX_CLEAN: now also C1029.C1, C509.C1, U1006.VOUT@0, U1006.VOUT@1; no longer C507.C1, C929.C1, U906.VOUT@0, U906.VOUT@1
- net 3V3_FB: now also R1010.1, R1011.2, U1002.FB@1; no longer R910.1, R911.2, U902.FB@1
- net 3V3_PGOOD: now also R1009.1, U1002.PG@1; no longer R909.1, U902.PG@1
- net 3V6_ANA: now also C1010.C1, C1013.C1, C1022.C1, C1023.C1, C1025.C1, L1002.2, R1007.2, U1001.SNS, U1005.EN, U1005.VIN, U1006.EN, U1006.VIN@0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; no longer C910.C1, C912.C1, C922.C1, C923.C1, C925.C1, L902.2, R907.2, U901.SNS, U905.EN, U905.VIN, U906.EN, U906.VIN@0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
- net 3V6_ANA_FB: now also R1007.1, R1008.2, U1001.FB; no longer R907.1, R908.2, U901.FB
- net 3V6_ANA_PGOOD: now also R1006.1, U1001.PG; no longer R906.1, U901.PG
- net 5V0: now also C1001.C1, C1002.C1, C1003.C1, C1004.C1, C1011.C1, C1014.C1, C1017.C1, C1018.C1, C1019.C1, L1003.2, L1005.1, U1001.EN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; no longer C901.C1, C902.C1, C903.C1, C904.C1, C911.C1, C914.C1, C917.C1, C918.C1, C919.C1, L903.2, L905.1, U901.EN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
- net 5V0_ANA_TXMIXER_CLEAN: now also C1020.C1, C1021.C1, L1005.2, U1003.VIN; no longer C920.C1, C921.C1, L905.2, U903.VIN
- net 5V0_ANA_TXPA_CLEAN: now also C1026.C1, C514.C1, U1003.VOUT; no longer C510.C1, C926.C1, U903.VOUT
- net DSP_D+: now also D1001.4, USB1001.D+; no longer D901.4, USB901.D+
- net DSP_D-: now also D1001.3, USB1001.D-; no longer D901.3, USB901.D-
- net DSP_ERASE: now also SJ1.1
- net DSP_MAIN_CLK: now also R906.1; no longer R809.1
- net FPGA_DDC_CLK: now also R905.1; no longer R805.1
- net FPGA_GP_CLK1: now also R907.1; no longer R807.1
- net FPGA_GP_CLK2: now also R904.1; no longer R804.1
- net FPGA_GP_CLK3: now also R908.1; no longer R808.1
- net GND: now also C1001.C2, C1002.C2, C1003.C2, C1004.C2, C1005.C2, C1006.C2, C1007.C2, C1008.C2, C1009.C2, C1010.C2, C1011.C2, C1012.C2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; no longer C415.C1, C417.C2, C419.C2, C429.C2, C508.C2, C515.C1, C802.C2, C803.C2, C804.C2, C805.C2, C807.C2, C808.C2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
- net N$10: now also C429.C2, R413.2, R415.2; no longer C427.C2, R409.2, R411.2
- net N$11: now also R907.2, U902.CLK1; no longer R807.2, U802.CLK1
- net N$12: now also R905.2, U902.CLK2; no longer R805.2, U802.CLK2
- net N$13: now also R908.2, U902.CLK3; no longer R808.2, U802.CLK3
- net N$14: now also R909.2, U902.CLK5; no longer R806.2, U802.CLK5
- net N$15: now also C433.C2; no longer C431.C2
- net N$16: now also C432.C2, C433.C1; no longer C430.C2, C431.C1
- net N$17: now also C432.C1; no longer C430.C1
- net N$19: now also R906.2, U902.CLK6; no longer R809.2, U802.CLK6
- net N$2: now also R506.1; no longer R502.1
- net N$22: now also C423.C1, R409.2; no longer C421.C1, R406.2
- net N$27: now also C431.C1, R414.2; no longer C429.C1, R410.2
- net N$3: now also R407.1, R412.1; no longer R405.1, R408.1
- net N$37: now also L1004.1, U1002.SW@1; no longer L904.1, U902.SW@1
- net N$4: now also C430.C1; no longer C428.C1
- net N$40: now also C1012.C1, U1002.SS@1; no longer C913.C1, U902.SS@1
- net N$41: now also C1008.C1, U1002.SS@0; no longer C908.C1, U902.SS@0
- net N$43: now also L1001.2, U1002.SW@0; no longer L901.2, U902.SW@0
- net N$47: now also R1001.2, USB1001.CC2; no longer R901.2, USB901.CC2
- net N$49: now also R1002.2, USB1001.CC1; no longer R902.2, USB901.CC1
- net N$5: now also R406.1, R411.2; no longer R404.1, R407.2
- net N$57: now also C511.C2, R507.2; no longer C509.C2, R503.2
- net N$58: now also F1001.2, USB1001.VBUS; no longer F901.2, USB901.VBUS
- net N$6: now also C508.C2, C511.C1, R506.2; no longer C506.C2, C509.C1, R502.2
- net N$60: now also U901.CLK, U902.CLKIN; no longer U801.CLK, U802.CLKIN
- net N$61: now also C906.C1, U902.XB, X901.2; no longer C807.C1, U802.XB, X801.2
- net N$62: now also C903.C1, U902.XA, X901.1; no longer C804.C1, U802.XA, X801.1
- net N$63: now also C515.C2; no longer C513.C2
- net N$64: now also C508.C1; no longer C506.C1
- net N$65: now also L1002.1, U1001.SW; no longer L902.1, U901.SW
- net N$66: now also C1005.C1, U1001.SS; no longer C905.C1, U901.SS
- net N$67: now also R604.1; no longer R603.1
- net N$69: now also R604.2; no longer R603.2
- net N$7: now also R904.2, U902.CLK0; no longer R804.2, U802.CLK0
- net N$73: now also C517.C2, R509.1; no longer C515.C2, R505.1
- net N$74: now also C516.C1, R508.2; no longer C514.C1, R504.2
- net N$75: now also C521.C2; no longer C519.C2
- net N$76: now also C520.C1; no longer C518.C1
- net N$77: now also C505.C1; no longer C504.C1
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