File: pcb/icyradio.brd (EAGLE design)
At the start: 150 x 100 mm, 386 parts, among them CON301 FPC-40P, J701 TRSJACK, J702 TRSJACK, J703 TRSJACK, Q801 AO3400, Q802 AO3400, U1001 MIC23155, U1002 MIC23159, U1003 MIC2019, U1004 ADP150UJZ-1.8, U1005 ADP150UJZ-3.3, U1006 MIC94305, U1007 MIC94305, U101 EFM32GG11B420F2048GL112, U201 ATSAMS70Q21B-C, U301 ICE40HX8K-CT256, U302 SST26VF064B, U401 DSC1211DE3-C0017, U402 LTC2206, U403 RT820T2, U501 ADL5385, U502 AD9117, U503 ADL5601, U601 DSC1201DE3-50M00000, U602 ADF4351, U701 TSCS25A3X1NDGXZAX, U702 CP2615, U801 ER-TFT035-6, U901 DSC1201DE3-50M00000, U902 SI5351C, X101 32.768 kHz, X401 DNP, X901 DNP

Commit message: Production ready, ordered
Parts:
- removed R717, R718, R720, R721: 600 Ohms, Resistor:RES0603
- removed R719, R722: 3.57 Ohms, Resistor:RES0603
- added L701, L702, L703, L704, L705, L706: 600 Ohms, Inductor:IND0603
- R603: value 5.1K Ohm -> 5.1K Ohms
- U403: value RT820T2 -> R820T2
Connections:
- net CODEC_HP_L: now also L704.1; no longer R722.1
- net CODEC_HP_R: now also L703.1; no longer R719.1
- net CODEC_LINE_L: now also L706.1; no longer R721.1
- net CODEC_LINE_R: now also L702.1; no longer R718.1
- net CODEC_MIC_L: now also L705.1; no longer R720.1
- net CODEC_MIC_R: now also L701.1; no longer R717.1
- net N$38: now also L701.2; no longer R717.2
- net N$39: now also L705.2; no longer R720.2
- net N$42: now also L702.2; no longer R718.2
- net N$44: now also L706.2; no longer R721.2
- net N$50: now also L704.2; no longer R722.2
- net N$54: now also L703.2; no longer R719.2

Commit message: Forgot to connect DAC common-mode, easy hardware fix tho
Parts:
- R509, R510, R511, R512: value 50 Ohms -> 49.9 Ohms
Connections:
- net GND: now also U502.20, U502.31
Changed lines of the file:
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@@
 <attribute name="VALUE" x="27.232" y="74.5456" size="0.8" layer="27" font="vector" ratio="10" rot="SR90" align="center-left"/>
 </element>
-<element name="R509" library="Resistor" package="RES0603" value="50 Ohms" x="26.1" y="70.3" smashed="yes" rot="R180">
+<element name="R509" library="Resistor" package="RES0603" value="49.9 Ohms" x="26.1" y="70.3" smashed="yes" rot="R180">
 <attribute name="NAME" x="24.5456" y="67.916" size="0.8" layer="25" font="vector" ratio="10" rot="SR0" align="center-left"/>
 <attribute name="TOLERANCE" value="" x="26.1" y="70.3" size="1.778" layer="27" rot="R180" display="off"/>
 <attribute name="VALUE" x="29.5544" y="72.332" size="0.8" layer="27" font="vector" ratio="10" rot="SR180" align="center-left"/>
 </element>
-<element name="R510" library="Resistor" package="RES0603" value="50 Ohms" x="22.5" y="70.3" smashed="yes" rot="R180">
+<element name="R510" library="Resistor" package="RES0603" value="49.9 Ohms" x="22.5" y="70.3" smashed="yes" rot="R180">
 <attribute name="NAME" x="21.2456" y="67.916" size="0.8" layer="25" font="vector" ratio="10" rot="SR0" align="center-left"/>
 <attribute name="TOLERANCE" value="" x="22.5" y="70.3" size="1.778" layer="27" rot="R180" display="off"/>
@@
 <attribute name="VALUE" x="33.432" y="74.5456" size="0.8" layer="27" font="vector" ratio="10" rot="SR90" align="center-left"/>
 </element>
-<element name="R511" library="Resistor" package="RES0603" value="50 Ohms" x="30.5" y="70.3" smashed="yes">
+<element name="R511" library="Resistor" package="RES0603" value="49.9 Ohms" x="30.5" y="70.3" smashed="yes">
 <attribute name="NAME" x="29.5456" y="67.916" size="0.8" layer="25" font="vector" ratio="10" rot="SR0" align="center-left"/>
 <attribute name="TOLERANCE" value="" x="30.5" y="70.3" size="1.778" layer="27" display="off"/>
 <attribute name="VALUE" x="27.0456" y="68.268" size="0.8" layer="27" font="vector" ratio="10" rot="SR0" align="center-left"/>
 </element>
-<element name="R512" library="Resistor" package="RES0603" value="50 Ohms" x="34.1" y="70.3" smashed="yes">
+<element name="R512" library="Resistor" package="RES0603" value="49.9 Ohms" x="34.1" y="70.3" smashed="yes">
 <attribute name="NAME" x="32.6456" y="67.916" size="0.8" layer="25" font="vector" ratio="10" rot="SR0" align="center-left"/>
 <attribute name="TOLERANCE" value="" x="34.1" y="70.3" size="1.778" layer="27" display="off"/>
@@
 <via x="73.9" y="52.05" extent="1-16" drill="0.2"/>
 <via x="73.4" y="51.55" extent="1-16" drill="0.2"/>
+<contactref element="U502" pad="20"/>
+<contactref element="U502" pad="31"/>
 </signal>
 <signal name="3V3">
