File: pcb/lna/icyradio-lna.brd (EAGLE design)
At the start: 30 x 20 mm, 15 parts, among them U1 ADL5601

Commit message: Sync library updates on LNA PCB
Connections:
- net GND: now also D1.C; no longer D1.1
- net N$146: now also D1.A; no longer D1.2

Commit message: Added CP2615 code Misc software changes Sync libraries
Parts:
- turned RFCON1 to 270 degrees
Changed lines of the file:
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@@
 <?xml version="1.0" encoding="utf-8"?>
 <!DOCTYPE eagle SYSTEM "eagle.dtd">
-<eagle version="9.5.1">
+<eagle version="9.6.1">
 <drawing>
 <settings>
@@
 <attribute name="VALUE" x="5.7456" y="15.968" size="0.8" layer="27" font="vector" ratio="10" rot="SR0" align="center-left"/>
 </element>
-<element name="RFCON1" library="RF Connector" package="SMA-EDGE" value="RFCON-SMA-EDGE" x="3.3" y="10" smashed="yes" rot="R90">
-<attribute name="NAME" x="5.47" y="5.99" size="0.8" layer="25" font="vector" ratio="10" rot="R180" align="center-left"/>
+<element name="RFCON1" library="RF Connector" package="SMA-EDGE" value="RFCON-SMA-EDGE" x="3.3" y="10" smashed="yes" rot="R270">
+<attribute name="NAME" x="1.13" y="14.01" size="0.8" layer="25" font="vector" ratio="10" align="center-left"/>
 </element>
 <element name="RFCON2" library="RF Connector" package="SMA-EDGE" value="RFCON-SMA-EDGE" x="26.7" y="10" smashed="yes" rot="R90">
