File: pcb/main/icyradio-main.brd (EAGLE design)
At the start: 167.7 x 111.2 mm, 492 parts, among them CON1101 2EDG-2P-5MM, CON201 FPC-22P, CON801 PCIE-X4-EDGE, J201 RJ45_MAG_LED_1G-TE-1-2301994-0, J701 TRSJACK, J702 TRSJACK, J703 TRSJACK, M701 SPH0641LM4H-1, M702 SPH0641LM4H-1, T601 UWB1-85E, T602 UWB1-85E, T603 UWB1-85E, T604 UWB1-85E, T605 UWB1-85E, T606 UWB1-85E, T607 UWB1-85E, T608 UWB1-85E, U1 DSC1203DA3-333M3333, U1001 74LVC1G157, U1002 DSB321SDA, U1003 SI5351C-B-GM, U101 SST26VF064B, U102 EFM32GG11B420F2048GL112, U103 SST26VF064B, U1102 MIC23159, U1201 ADM7172ACPZ-5.0, U1202 ADM7171ACPZ-1.3, U1203 ADM7171ACPZ-1.3, U1204 MIC23159, U1205 MIC5166, U1206 MIC23155, U1208 ADP7142AUJZ-3.3, U1209 ADP150UJZ-1.8, U2 LT7182S, U201 MIC2019, U202 RPI-CM4, U301 XC7A100TFGG484, U401 MT41K256M16TW-125, U402 MT41K256M16TW-125, U501 AD9361, U502 LTC6957-3, U503 TG2520SMN-40.0000M, U601 MIC2019, U602 MIC2019, U603 MIC2019, U604 MIC2019, U605 ADL5601, U606 ADL5601, U701 ADAU1372, U901 CYUSB3014, X101 32.768 kHz, X901 30MHz

Commit message: Work on PCB
Signed-off-by: João Silva <jgc3silva@gmail.com>
Parts:
- added C10, C11, C12, C13, C14: 22uF, Capacitor:CAP0603
- added C16: 100nF, Capacitor:CAP0402
- added R10, R11: 49.9 Ohms, Resistor:RES0402
- added R12, R13, R14, R15: 1K Ohms, Resistor:RES0402
- added RFCON1, RFCON2: RFCON-SMA, RF Connector:SMA
- added U3: 8V97003, Renesas:VFQFPN48
Connections:
- new net N$43: C10.1, U3.11
- new net N$75: C14.1, U3.32
- new net N$76: C13.1, U3.4
- new net N$77: C12.1, U3.35
- new net N$84: C11.1, U3.1
- new net N$85: R10.1, U3.45
- new net N$86: R11.1, U3.46
- new net N$88: C16.2, R12.1, R13.2, U3.22
- new net N$89: R14.1, R15.2, U3.23
- net GND: now also C10.2, C11.2, C12.2, C13.2, C14.2, R13.1, R15.1, RFCON1.GND@0, RFCON1.GND@1, RFCON1.GND@2, RFCON1.GND@3, RFCON2.GND@0, RFCON2.GND@1, RFCON2.GND@2, RFCON2.GND@3, U3.14, U3.17, U3.19, U3.20, U3.38, U3.41, U3.44, U3.47, U3.49

Commit message: PCB Work
Signed-off-by: João Silva <jgc3silva@gmail.com>
Parts:
- removed C1: 10uF, Capacitor:CAP1206
- removed C10, C11, C12, C13, C14: 22uF, Capacitor:CAP0603
- removed C1109, C1126, C1227, C1232, C2, C4, C6: 1uF, Capacitor:CAP0603
- removed C1112, C1117, C1233: 470pF, Capacitor:CAP0603
- removed C1114, C1115, C1119, C1124, C1224, C1228, C1229, C1241, C1243, C1244, C5, C707, C709, C710, C711, C712: 100nF, Capacitor:CAP0603
- removed C1121, C1123: 100uF, Capacitor:CAP1206
- removed C1249, C9: 4.7uF, Capacitor:CAP0402
- removed C1251, C1253, C713: 47uF, Capacitor:CAP0603
- removed C16: 100nF, Capacitor:CAP0402
- removed C3: 4.7uF, Capacitor:CAP0603
- removed C7, C708, C8: 10uF, Capacitor:CAP0603
- removed C719, C720: DNP, Capacitor:CAP0603
- removed D1104: SK54L, Generic Diode:DO214AA
- removed L1: 1.5uH, Inductor:IND0404
- removed L1103: 4.7uH, Inductor:IND0404
- removed R10, R11: 49.9 Ohms, Resistor:RES0402
- removed R1008, R1009, R1010, R1011, R1012, R9: 0 Ohms, Resistor:RES0603
- removed R1113, R1115, R2, R3, R4, R8, R906, R907: 10K Ohms, Resistor:RES0603
- removed R1116: 309K Ohms, Resistor:RES0603
- removed R1117: 71.5K Ohms, Resistor:RES0603
- removed R12, R13, R14, R15: 1K Ohms, Resistor:RES0402
- removed R5: 36.5K Ohms, Resistor:RES0603
- removed R6: 124K Ohms, Resistor:RES0603
- removed R7: 51.1K Ohms, Resistor:RES0603
- removed R707, R709, R711: 49.9K Ohms, Resistor:RES0603
- removed R708, R710: 2.21K Ohms, Resistor:RES0603
- removed R904: 50K Ohms, Resistor:RES0603
- removed R905: 100K Ohms, Resistor:RES0603
- removed RFCON1, RFCON2: RFCON-SMA, RF Connector:SMA
- removed U1002: DSB321SDA, Crystal:TCXO-3225
- removed U2: LT7182S, Analog Devices:LQFN40_ASYM_CORNER
- removed U3: 8V97003, Renesas:VFQFPN48
- removed U901: CYUSB3014, Cypress:BGA121
- removed X901: 30MHz, Crystal:4-SMD-3225
- added C1009: 10uF, Capacitor:CAP1206
- added C1010, C1101, C1301, C1302, C1303, C1304, C1309, C1315, C1324, C1328, C1329, C1333, C1336, C1341, C1343, C1344, C1346, C1349, C911, C912: 100nF, Capacitor:CAP0402
- added C1305, C1335, C404: 4.7uF, Capacitor:CAP0603
- added C1306, C1307, C1308: 10nF, Capacitor:CAP0402
- added C1310: 100uF, Capacitor:CAP1206
- added C1311, C1322, C1334, C1340, C1345: 470pF, Capacitor:CAP0402
- added C1312, C1313, C1314, C1316, C1317, C1318, C1319, C1320, C1321: 10uF, Capacitor:CAP0603
- added C1327, C1332, C913: 1uF, Capacitor:CAP0402
- added C819, C820: DNP, Capacitor:CAP0402
- added D1001: SP3004-04XTG, TVS:SOT563
- added L1301, L1302: 2.2uH, Inductor:IND3515
- added R1103, R1208, R1211, R1301, R1304, R1308, R1313, R1316: 10K Ohms, Resistor:RES0402
- added R1104, R1306: 100K Ohms, Resistor:RES0402
- added R1105, R1215: 0 Ohms, Resistor:RES0402
- added R1212: 36.5K Ohms, Resistor:RES0402
- added R1213: 124K Ohms, Resistor:RES0402
- added R1302: 301K Ohms, Resistor:RES0402
- added R1303: 158K Ohms, Resistor:RES0402
- added R1305: 118K Ohms, Resistor:RES0402
- added R1307: 10K Ohms, Resistor:RES0603
- added R1309: 324K Ohms, Resistor:RES0402
- added R1310: 107K Ohms, Resistor:RES0402
- added R1311: 274K Ohms, Resistor:RES0603
- added R1312: 294K Ohms, Resistor:RES0603
- added R1314: 309K Ohms, Resistor:RES0402
- added R1315: 71.5K Ohms, Resistor:RES0402
- added R428: 240 Ohms, Resistor:RES0402
- added R804, R806, R808, R810: 2.21K Ohms, Resistor:RES0402
- added R805, R807, R809, R811: 49.9K Ohms, Resistor:RES0402
- added RFCON701, RFCON702: RFCON-SMA, RF Connector:SMA
- added U1101: 74LVC1G157, Logic:SC70-6
- added U1301: ADM7172ACPZ-5.0, Analog Devices:LFCSP8_3X3
- added U1307: MIC23159, Microchip:VQFN20
- added U801: ADAU1372, Analog Devices:QFN40
- added X1001: 30MHz, Crystal:4-SMD-3225
- C1001, C1002, C1003, C1004, C1005, C1006, C101, C102, C103, C104, C105, C106, C107, C108, C109, C110, C1103, C1106, C111, C112, C114, C115, C1201, C1202, C201, C203, C204, C301, C302, C303, C304, C305, C306, C307, C308, C309, C310, C311, C312, C313, C314, C315, C316, C317, C318, C501, C502, C503, C504, C505, C506, C507, C508, C509, C511, C512, C513, C514, C515, C516, C517, C518, C519, C520, C521, C522, C523, C524, C525, C526, C527, C528, C605, C606, C607, C608, C625, C626, C627, C628, C629, C638, C639, C640, C641, C642, C643, C644, C645, C646, C647, C648, C910: device Capacitor:CAP0603 -> Capacitor:CAP0402
- C1007, C1008: value 10pF -> 18pF; device Capacitor:CAP0603 -> Capacitor:CAP0402
- C1102, C909: value 10uF -> 100nF; device Capacitor:CAP1206 -> Capacitor:CAP0402
- C1104, C1105, C403: value 4.7uF -> 100nF; device Capacitor:CAP0603 -> Capacitor:CAP0402
- C1107: value 1uF -> 10pF; device Capacitor:CAP0603 -> Capacitor:CAP0402
- C1108: value 100nF -> 10pF; device Capacitor:CAP0603 -> Capacitor:CAP0402
- C1203, C1204: value 100nF -> 10uF; device Capacitor:CAP0603 -> Capacitor:CAP1206
- C1205: value 4.7uF -> 10uF
- C1206: value 10nF -> 4.7uF; device Capacitor:CAP0603 -> Capacitor:CAP0402
- C1207: value 10nF -> 1uF; device Capacitor:CAP0603 -> Capacitor:CAP0402
- C1208: value 10nF -> 4.7uF
- C1209: value 100nF -> 4.7uF
- C1210: value 100uF -> 1uF; device Capacitor:CAP1206 -> Capacitor:CAP0603
- C1211: value 470pF -> 1uF
- C1212, C1213: value 10uF -> 100nF
- C1214, C1221: value 10uF -> 1uF
- C1215: value 100nF -> 1uF
- C1216, C1219: value 10uF -> 100uF; device Capacitor:CAP0603 -> Capacitor:CAP1206
- C1217: value 10uF -> 4.7uF; device Capacitor:CAP0603 -> Capacitor:CAP0402
- C1220: value 10uF -> 47uF
- C1222: value 470pF -> 47uF
- C701: value 10uF -> 100nF; device Capacitor:CAP0603 -> Capacitor:CAP0402
- C702, C703, C704, C705: value 100nF -> 22uF
- C706: value 10uF -> 22uF
- C801, C806: value 0 Ohms -> 10uF; device Capacitor:CAP0201 -> Capacitor:CAP0603
- C802, C803, C804, C805: value 0 Ohms -> 100nF; device Capacitor:CAP0201 -> Capacitor:CAP0402
- C807, C809, C810, C811, C812: device Capacitor:CAP0201 -> Capacitor:CAP0402
- C808: value 100nF -> 10uF; device Capacitor:CAP0201 -> Capacitor:CAP0603
- C813: value 1uF -> 47uF; device Capacitor:CAP0402 -> Capacitor:CAP0603
- C901, C902, C903, C904, C905, C906: value 100nF -> 0 Ohms; device Capacitor:CAP0603 -> Capacitor:CAP0402
- C907, C908: value 18pF -> 100nF; device Capacitor:CAP0603 -> Capacitor:CAP0402
- D901: value SP3004-04XTG -> SK54L; device TVS:SOT563 -> Generic Diode:DO214AA
- L1201: value 2.2uH -> 4.7uH; device Inductor:IND3515 -> Inductor:IND0404
- L1202: value 2.2uH -> 1.5uH; device Inductor:IND3515 -> Inductor:IND0404
- R1001: value 10K Ohms -> 330 Ohms; device Resistor:RES0603 -> Resistor:RES0402
- R1002, R101, R102, R103, R104, R105, R106, R107, R108, R109, R110, R111, R112, R113, R1207, R201, R202, R203, R204, R205, R301, R302, R502, R503, R504, R601, R602, R603, R604, R605, R606, R607, R608, R609, R610, R611, R612, R613, R614, R615, R616, R801: device Resistor:RES0603 -> Resistor:RES0402
- R1003: value 10K Ohms -> 1.6K Ohms; device Resistor:RES0603 -> Resistor:RES0402
- R1004: value 100K Ohms -> 50K Ohms; device Resistor:RES0603 -> Resistor:RES0402
- R1005: value 0 Ohms -> 100K Ohms; device Resistor:RES0603 -> Resistor:RES0402
- R1006, R1007: value 0 Ohms -> 10K Ohms; device Resistor:RES0603 -> Resistor:RES0402
- R1101: value 1K Ohms -> 10K Ohms; device Resistor:RES0603 -> Resistor:RES0402
- R1102: value 1K Ohms -> 100K Ohms; device Resistor:RES0603 -> Resistor:RES0402
- R1106, R1111: value 100K Ohms -> 0 Ohms; device Resistor:RES0603 -> Resistor:RES0402
- R1107, R1108, R1112: value 10K Ohms -> 0 Ohms; device Resistor:RES0603 -> Resistor:RES0402
- R1109: value 324K Ohms -> 0 Ohms; device Resistor:RES0603 -> Resistor:RES0402
- R1110: value 107K Ohms -> 0 Ohms; device Resistor:RES0603 -> Resistor:RES0402
- R1201: value 10K Ohms -> 100K Ohms
- R1202: value 301K Ohms -> 10K Ohms
- R1203: value 158K Ohms -> 100K Ohms
- R1205: value 118K Ohms -> 1K Ohms; device Resistor:RES0603 -> Resistor:RES0402
- R1206: value 100K Ohms -> 1K Ohms; device Resistor:RES0603 -> Resistor:RES0402
- R1209: value 274K Ohms -> 10K Ohms; device Resistor:RES0603 -> Resistor:RES0402
- R1210: value 294K Ohms -> 10K Ohms; device Resistor:RES0603 -> Resistor:RES0402
- R1214: value 10K Ohms -> 51.1K Ohms; device Resistor:RES0603 -> Resistor:RES0402
- R401, R402, R403, R404, R405, R406, R407, R408, R410, R411, R412, R413, R414, R415, R416, R417, R418, R419, R420, R421, R422, R423, R424, R425: value 120 Ohms -> 40.2 Ohms
- R426: value 240 Ohms -> 40.2 Ohms
- R427: value 80.6 Ohms -> 40.2 Ohms
- R701: value 10K Ohms -> 1K Ohms; device Resistor:RES0603 -> Resistor:RES0402
- R702, R703: value 49.9K Ohms -> 1K Ohms; device Resistor:RES0603 -> Resistor:RES0402
- R704: value 2.21K Ohms -> 1K Ohms; device Resistor:RES0603 -> Resistor:RES0402
- R705: value 49.9K Ohms -> 49.9 Ohms; device Resistor:RES0603 -> Resistor:RES0402
- R706: value 2.21K Ohms -> 49.9 Ohms; device Resistor:RES0603 -> Resistor:RES0402
- R802, R803: value 10K Ohms -> 49.9K Ohms; device Resistor:RES0603 -> Resistor:RES0402
- R901: value 330 Ohms -> 10K Ohms; device Resistor:RES0603 -> Resistor:RES0402
- R902: value 100K Ohms -> 10K Ohms; device Resistor:RES0603 -> Resistor:RES0402
- R903: value 1.6K Ohms -> 10K Ohms; device Resistor:RES0603 -> Resistor:RES0402
- U1001: value 74LVC1G157 -> CYUSB3014; device Logic:SC70-6 -> Cypress:BGA121
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- renumbered C1110 to C1338, C1120 to C1347, C1127 to C1351, C1223 to C1323, C1225 to C1325, C1226 to C1326, C1230 to C1330, C1231 to C1331, C1237 to C1337, C1238 to C1339, C1242 to C1342, C1250 to C1348, C1252 to C1350, C714 to C814, C715 to C815, C716 to C816, C717 to C817, C718 to C818, C721 to C821, C722 to C822, CON1101 to CON1201, CON801 to CON901, D1 to D1205, D1101 to D1201, D1102 to D1202, D1103 to D1204, D1105 to D1203, F1101 to F1201, F901 to F1001, FB701 to FB801, J701 to J801, J702 to J802, J703 to J803, L1101 to L1304, L1102 to L1305, L1203 to L1303, L701 to L801, L702 to L802, L901 to L1001, M701 to M801, M702 to M802, R1 to R429, RFCON1001 to RFCON1101, RFCON1002 to RFCON1102, U1 to U403, U1003 to U1103, U1202 to U1302, U1203 to U1303, U1204 to U1304, U1205 to U1305, U1206 to U1306, U1208 to U1308, U1209 to U1309, USB901 to USB1001
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Connections:
- new net N$87: C401.1, R410.1, R418.2
- net !1V0_FAULT: now also R1210.1, U1201.27; no longer R4.1, U2.27
- net !5V0_FAULT: now also R1209.1, U1201.28; no longer R2.1, U2.28
- net !CLK_MNGR_IRQ: now also R1104.1; no longer R1004.1
- net !CLK_MNGR_OE: now also R1102.1; no longer R1002.1
- net !CODEC_RST: now also R801.2, U801.27; no longer R701.2, U701.27
- net !DDR3_CAS: now also R420.1; no longer R418.1
- net !DDR3_CS: now also R421.1; no longer R419.1
- net !DDR3_RAS: now also R425.1; no longer R423.1
- net !DDR3_WE: now also R424.1; no longer R422.1
- net !FIFO_RESET: now also R1002.2; no longer R902.2
- net !PCIE_SLOT_CLK_REQ: now also R901.1; no longer R801.1
- net !PCIE_SLOT_RST: now also C913.1, R903.1; no longer C813.1, R803.1
- net !PCIE_SLOT_WAKE: now also R902.1; no longer R802.1
- net 0V675_DDR3_VREF: now also C1332.1; no longer C1232.1
- net 0V675_DDR3_VTT: now also C401.2, C404.1, R417.1, R426.2, R427.2; no longer C401.1, R410.1, R417.2, R418.2
- net 12V0: now also R1203.2; no longer R1111.2
- net 12V0_VSENSE: now also C1202.1, R1203.1, R1204.2; no longer C1114.1, R1111.1, R1112.2
- net 1V0: now also C1217.1, C1220.1, C1222.1, L1202.2, U1201.11; no longer C1249.1, C1251.1, C1253.1, L1.2, U2.11
- net 1V0_BOOST: now also C1213.2, U1201.13; no longer C5.2, U2.13
- net 1V0_PGOOD: now also R1208.1, U1201.32; no longer R3.1, U2.32
- net 1V0_SW: now also C1213.1, L1202.1, U1201.16, U1201.17, U1201.44; no longer C5.1, L1.1, U2.16, U2.17, U2.44
- net 1V2: now also C1341.1, R1311.2; no longer C1241.1, R1209.2
- net 1V2_FB: now also R1311.1, R1312.2; no longer R1209.1, R1210.2
- net 1V2_PGOOD: now also R1307.1; no longer R1207.1
- net 1V2_SS: now also C1334.1; no longer C1233.1
- net 1V35: now also C1324.1, L1302.2, R1305.2; no longer C1224.1, L1202.2, R1205.2
- net 1V35_FB: now also R1305.1, R1306.2; no longer R1205.1, R1206.2
- net 1V35_PGOOD: now also R1304.1; no longer R1204.1
- net 1V35_SS: now also C1322.1; no longer C1222.1
- net 1V35_SW: now also L1302.1; no longer L1202.1
- net 1V3_TRX: now also C1314.1, C1317.1, C1319.1, C1321.1; no longer C1214.1, C1217.1, C1219.1, C1221.1
- net 1V3_TRX_LO_SYNTH: now also C1313.1, C1316.1, C1318.1, C1320.1; no longer C1213.1, C1216.1, C1218.1, C1220.1
- net 1V8: now also C1309.1, C1310.1, L1301.1, R1302.2; no longer C1209.1, C1210.1, L1201.1, R1202.2
- net 1V8_FB: now also R1302.1, R1303.2; no longer R1202.1, R1203.2
- net 1V8_PGOOD: now also R1301.1; no longer R1201.1
- net 1V8_SS: now also C1311.1; no longer C1211.1
- net 1V8_SW: now also L1301.2; no longer L1201.2
- net 1V8_VIN_REG_VDD: now also C1206.1, U1201.7; no longer C9.1, U2.7
- net 2V5: now also C1303.1, C1304.1, C1336.1, C1344.1, R1308.2, R1309.2, U1307.17; no longer C1108.1, C1203.1, C1204.1, C1244.1, R1108.2, R1109.2, U1102.17
- net 2V5_FB: now also R1309.1, R1310.2, U1307.16; no longer R1109.1, R1110.2, U1102.16
- net 2V5_PGOOD: now also R1308.1, U1307.15; no longer R1108.1, U1102.15
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Routing:
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
Commit message: Work on schematic
Signed-off-by: João Silva <jgc3silva@gmail.com>
Parts:
- removed C1009: 10uF, Capacitor:CAP1206
- removed C1010, C1104, C1105, C1106, C302, C303, C304, C305, C306, C307, C308, C309, C310, C311, C312, C313, C314, C315, C316, C317, C318: 100nF, Capacitor:CAP0402
- removed C1107, C1108: 10pF, Capacitor:CAP0402
- removed D1001: SP3004-04XTG, TVS:SOT563
- removed D101: LED0603, LED:0603
- removed D301: B0530W, Generic Diode:SOD-123
- removed D901: SK54L, Generic Diode:DO214AA
- removed R106, R110, R112: 4.7K Ohms, Resistor:RES0402
- removed R109, R111: 330 Ohms, Resistor:RES0402
- removed R1105, R1106, R1107: 0 Ohms, Resistor:RES0402
- removed R113, R301: 10K Ohms, Resistor:RES0402
- removed R302: 100K Ohms, Resistor:RES0402
- removed TC101: TC2050-IDC, TagConnect:TC2050-IDC
- removed U101, U103: SST26VF064B, Microchip:WSOIC8
- removed U102: EFM32GG11B420F2048GL112, EFM32:BGA112
- removed USB1001: USB3-B-TH-FLAT-SIDE, USB Connector:USB3-B-TH-FLAT-SIDE
- removed X1001: 30MHz, Crystal:4-SMD-3225
- removed X101: 32.768 kHz, Crystal:2-SMD-3215
- added C1, C11, C12, C121, C122, C124, C125, C13, C14, C15, C16, C17, C18, C19, C2, C20, C21, C22, C23, C24, C25, C26, C27, C28, C29, C3, C30, C31, C32, C33, C34, C35, C36, C37, C38, C39, C4, C40, C41, C42, C43, C44, C45, C46, C47, C48, C49, C50, C53, C54, C55, C56: 100nF, Capacitor:CAP0402
- added C10, C7, C8, C9: 1uF, Capacitor:CAP0402
- added C100, C116, C117, C118, C58, C60, C61, C62, C63, C64, C65, C66, C75, C76, C77, C78, C79, C80, C81, C86, C87, C88, C91, C92, C93, C94, C97, C98, C99: 470nF, Capacitor:CAP0402
- added C119, C120, C1224, C123, C126, C67, C68, C69, C70, C71, C72, C73, C74, C82, C83, C84, C85, C89, C90, C95, C96: 4.7uF, Capacitor:CAP0402
- added C1223, C1225: 100uF, Capacitor:CAP1206
- added C1226, C1229: 47uF, Capacitor:CAP0603
- added C1227, C51, C52: 10uF, Capacitor:CAP0603
- added C1228: 1uF, Capacitor:CAP0603
- added C5, C6: 220pF, Capacitor:CAP0402
- added D1: B0530W, Generic Diode:SOD-123
- added Q1201, Q1203, Q1205: AO4805, Alpha Omega:SOIC8
- added Q1202, Q1204, Q1206: AO3400, Alpha Omega:SOT23
- added R1, R1218, R1219, R1221, R1222, R1223, R4, R5: 10K Ohms, Resistor:RES0402
- added R1216, R1217, R1220, R3: 1K Ohms, Resistor:RES0402
- added R1224: 36.5K Ohms, Resistor:RES0402
- added R1225: 124K Ohms, Resistor:RES0402
- added R1226: 51.1K Ohms, Resistor:RES0402
- added R1227: 0 Ohms, Resistor:RES0402
- added R2: TBD Ohms, Resistor:RES0402
- added R6: 100 Ohms, Resistor:RES0402
- added TC1101, TC301: TC2050-IDC, TagConnect:TC2050-IDC
- added TP1, TP2, TP4, TP5, TP6, TP7: TESTPOINT-0.7MM, PADs:PAD0.7MM
- added U1: MIC2019, Microchip:SOT23-6
- added U1202: LT7182S, Analog Devices:LQFN40_ASYM_CORNER
- added USB1101: USB-C-16P-SMD-FLAT-SIDE-TYPE-2, USB Connector:USB-C-16P-SMD-FLAT-SIDE-TYPE-2
- C1007, C1008: value 18pF -> 10pF
- C101, C102, C107, C108, C114: value 100nF -> 4.7uF
- C103, C104, C105, C106, C109, C110, C111, C301: value 100nF -> 470nF
- C112, C115: value 1uF -> 470nF
- C113: device Capacitor:CAP0603 -> Capacitor:CAP0402
- C1204: value 10uF -> 1uF; device Capacitor:CAP1206 -> Capacitor:CAP0603
- C1205: device Capacitor:CAP0603 -> Capacitor:CAP1206
- C1206: value 4.7uF -> 100nF
- C1207, C1327: value 1uF -> 100nF
- C1209: value 4.7uF -> 100nF; device Capacitor:CAP0603 -> Capacitor:CAP0402
- C1210, C1211: value 1uF -> 10uF; device Capacitor:CAP0603 -> Capacitor:CAP1206
- C1212: value 100nF -> 10uF; device Capacitor:CAP0603 -> Capacitor:CAP1206
- C1213: value 100nF -> 10uF
- C1214: value 1uF -> 4.7uF; device Capacitor:CAP0603 -> Capacitor:CAP0402
- C1215: value 1uF -> 4.7uF
- C1216: value 100uF -> 4.7uF; device Capacitor:CAP1206 -> Capacitor:CAP0603
- C1217: value 4.7uF -> 1uF; device Capacitor:CAP0402 -> Capacitor:CAP0603
- C1218: value 10uF -> 1uF
- C1219: value 100uF -> 100nF; device Capacitor:CAP1206 -> Capacitor:CAP0603
- C1220: value 47uF -> 100nF
- C1222: value 47uF -> 1uF
- C1328: value 100nF -> 1uF
- D1201, D1202: value LED0603 -> B0530W; device LED:0603 -> Generic Diode:SOD-123
- D1203: value SK54L -> B0530W; device Generic Diode:DO214AA -> Generic Diode:SOD-123
- D1204: value SMAJ20A -> LED0603; device TVS:DO214AC -> LED:0603
- D1205: value B0530W -> SMAJ20A; device Generic Diode:SOD-123 -> TVS:DO214AC
- L1201: device Inductor:IND0404 -> Coilcraft:XGL6030
- L1202: value 1.5uH -> 2.2uH; device Inductor:IND0404 -> Coilcraft:XGL6030
- L1301, L1302, L1303, L1304, L1305: device Inductor:IND3515 -> Coilcraft:XGL351X
- R1001: value 330 Ohms -> 10K Ohms
- R1003: value 1.6K Ohms -> 10K Ohms
- R1004: value 50K Ohms -> 100K Ohms
- R1005: value 100K Ohms -> 0 Ohms
- R1006, R1007: value 10K Ohms -> 0 Ohms
- R101, R102: value 100K Ohms -> 4.7K Ohms
- R105: value 4.7K Ohms -> 330 Ohms
- R1101: value 10K Ohms -> 330 Ohms
- R1102: value 100K Ohms -> 90.9K Ohms
- R1104: value 100K Ohms -> 10K Ohms
- R1205: value 1K Ohms -> 10K Ohms
- R1207: value 10K Ohms -> 1K Ohms
- R1208, R1210: value 10K Ohms -> 100K Ohms; device Resistor:RES0402 -> Resistor:RES0603
- R1209, R1211: device Resistor:RES0402 -> Resistor:RES0603
- R1212: value 36.5K Ohms -> 10K Ohms
- R1213: value 124K Ohms -> 1K Ohms
- R1214: value 51.1K Ohms -> 1K Ohms
- R1215: value 0 Ohms -> 10K Ohms
- U1001: value CYUSB3014 -> 74LVC1G157; device Cypress:BGA121 -> Logic:SC70-6
- U1101: value 74LVC1G157 -> UPD301C; device Logic:SC70-6 -> Microchip:VQFN40
- U1201: value LT7182S -> MCP1804-3302; device Analog Devices:LQFN40_ASYM_CORNER -> Microchip:SOT23-5
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- renumbered F1001 to F1101, L1001 to L1101, R1108 to R1008, R1109 to R1009, R1110 to R1010, R1111 to R1011, R1112 to R1012, RFCON1101 to RFCON1001, RFCON1102 to RFCON1002, U1102 to U1002, U1103 to U1003
Connections:
- removed net !FIFO_RESET: R1002.2
- removed net !FPGA_CRESET: R302.2, U102.G2
- removed net !FPGA_SMC_IRQ: U102.F2
- removed net !FPGA_SPI_CS: U102.H1
- removed net !SMC_QSPI_CS0: R102.1, U102.C2, U103.1
- removed net !SMC_QSPI_CS1: R101.1, U101.1, U102.C1
- removed net !SMC_RESET: R113.1, TC101.10, U102.K6
- removed net !TFT_SPI_CS: U102.J6
- removed net DSP_I2C_SCL: R104.1
- removed net DSP_I2C_SDA: R103.1
- removed net EXT_VIN_FUSED: D1203.A, D1204.C, F1201.1
- removed net FPGA_CBSEL1\: U102.G1
- removed net FPGA_CDONE: R301.1, U102.F1
- removed net FPGA_SPI_SCK: U102.J2
- removed net FPGA_SPI_SDI: U102.J1
- removed net FPGA_SPI_SDO: U102.H2
- removed net FPGA_VPP_FAST: TP3.TP
- removed net N$144: D101.A, R108.1
- removed net N$149: D1201.A, R1205.1
- removed net PCIE_SLOT_12V0: CON901.A2, CON901.A3, CON901.B1, CON901.B2, CON901.B3, D901.A
- removed net SMC_LED: R108.2, U102.B1
- removed net SMC_LFXTAL_N: U102.L1, X101.2
- removed net SMC_LFXTAL_P: U102.K1, X101.1
- removed net SMC_QSPI_CLK: U101.6, U102.A2, U103.6
- removed net SMC_QSPI_D0: U101.5, U102.D2, U103.5
- removed net SMC_QSPI_D1: U101.2, U102.D1, U103.2
- removed net SMC_QSPI_D2: U101.3, U102.E3, U103.3
- removed net SMC_QSPI_D3: U101.7, U102.E2, U103.7
- removed net SMC_SWCLK: TC101.4, U102.E8
- removed net SMC_SWDIO: TC101.2, U102.D8
- removed net SMC_SWO: TC101.6, U102.C8
- removed net SMC_USB_D_N: U102.A10
- removed net SMC_USB_D_P: U102.A11
- removed net SMC_VCORE: C115.1, U102.F11
- removed net TFT_SPI_MISO: U102.H5
- removed net TFT_SPI_MOSI: U102.H4
- removed net TFT_SPI_SCK: U102.J5
- removed net USB_RX_N: USB1001.8
- removed net USB_RX_P: USB1001.9
- removed net USB_TX_N: C1005.2
- removed net USB_TX_P: C1006.2
- removed net USB_VBUS: C1009.1, C1010.1, C112.1, D1001.5, F1101.1, R1004.2, R1205.2, U102.B8
- removed net VIN_REG_EXTVCC: C1207.1, D1205.C, U1201.21
- new net !PMC_RESET: R1104.1, TC1101.10, U1101.40
- new net 12V0_EN: Q1204.1, R1212.2
- new net 3V3_PM: C1.1, C1208.1, C1209.1, C2.1, C3.1, C4.1, R1104.2, TC1101.1, U1101.14, U1101.16, U1101.21, U1101.3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
- new net FPGA_TCK: TC301.4, U301.V12
- new net FPGA_TDI: R4.1, TC301.8, U301.R13
- new net FPGA_TDO: TC301.6, U301.U13
- new net FPGA_TMS: R5.1, TC301.2, U301.T13
- new net N$90: Q1205.2, Q1205.4, R1216.1, R1217.2
- new net N$91: Q1206.3, R1217.1
- new net N$92: C1204.1, D1201.C, D1202.C, D1203.C, U1201.1, U1201.4
- new net N$93: C8.1, U1101.5
- new net N$94: C9.1, D1.A, U1.6
- new net N$95: R2.2, U1.5
- new net PMC_SWCLK: TC1101.4, U1101.7
- new net PMC_SWDIO: TC1101.2, U1101.8
- new net PMC_SWO: TC1101.6
- new net USB_CC1: C6.1, U1101.4, USB1101.A5
- new net USB_CC2: C5.1, U1101.2, USB1101.B5
- new net VBUS: C1102.1, C1203.1, D1.C, D1201.A, F1101.1, Q1201.7, Q1201.8, R1102.2, R1210.2
- new net VBUS_SNK_EN: Q1202.1, R1205.2
- new net VBUS_SRC_EN: R1.2, U1.3
- new net VBUS_VSENSE: C1207.1, R1210.1, R1211.2
- new net VEXT: C1210.1, D1203.A, D1205.C, F1201.1, Q1205.7, Q1205.8, R1203.2
- new net VEXT_EN: Q1206.1, R1215.2
- new net VEXT_VSENSE: C1202.1, R1203.1, R1204.2
- net !1V0_FAULT: now also R1222.1, U1202.27; no longer R1210.1, U1201.27
- net !5V0_FAULT: now also R1221.1, U1202.28; no longer R1209.1, U1201.28
- net !CLK_MNGR_IRQ: now also R1004.1; no longer R1104.1
- net !CLK_MNGR_OE: now also R1002.1; no longer R1102.1
- net !DDR3_RESET: now also R3.2
- net !TRX_RESET: no longer U102.A4
- net !TRX_SPI_CS: no longer U102.B2
- net 0V675_DDR3_VREF: now also C11.1, C12.1, C13.1, C14.1, C53.1, C54.1, C55.1, C56.1, U301.E3, U301.N3, U301.V3, U301.W7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
- net 12V0: now also C1205.1, CON901.A2, CON901.A3, CON901.B1, CON901.B2, CON901.B3, D1202.A, Q1203.7, Q1203.8, R1208.2; no longer R1203.2
- net 12V0_VSENSE: now also C1206.1, R1208.1, R1209.2; no longer C1202.1, R1203.1, R1204.2
- net 1V0: now also C1224.1, C1226.1, C1229.1, C124.1, C125.1, C126.1, C58.1, C60.1, C61.1, C62.1, C63.1, C64.1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; no longer C1217.1, C1220.1, C1222.1, U1201.11
- net 1V0_BOOST: now also C1220.2, U1202.13; no longer C1213.2, U1201.13
- net 1V0_PGOOD: now also R1219.1, TP2.TP, U1202.32, U1306.2; no longer R1208.1, U1201.32
- net 1V0_SW: now also C1220.1, U1202.16, U1202.17, U1202.44; no longer C1213.1, U1201.16, U1201.17, U1201.44
- net 1V2: now also C121.1, C122.1, C123.1, R6.2, U301.B11, U301.B5, U301.B7, U301.B9, U301.C4, U301.C8; no longer C303.1, C306.1, C308.1, C310.1, C312.1, C314.1, C316.1, C318.1
- net 1V2_PGOOD: now also TP3.TP, U1304.18, U1307.18, U1307.9
- net 1V35: now also C109.1, C110.1, C111.1, C112.1, C113.1, C114.1, C115.1, C116.1, C117.1, C118.1, C119.1, C120.1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
- net 1V35_PGOOD: now also TP7.TP
- net 1V8: now also C77.1, C78.1, C79.1, C80.1, C81.1, C82.1, C83.1, C84.1, R1301.2, U301.E12, U301.H12, U301.K10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
- net 1V8_PGOOD: now also TP4.TP, U1304.9
- net 1V8_VIN_REG_VDD: now also C1214.1, U1202.7; no longer C1206.1, U1201.7
- net 2V5: now also C100.1, C101.1, C102.1, C103.1, C104.1, C105.1, C106.1, C107.1, C108.1, C97.1, C98.1, C99.1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; no longer C110.1, C302.1, C305.1, U102.D5
- net 2V5_PGOOD: now also TP5.TP
- net 3V0_VIN_REG_INTVCC: now also C1213.1, U1202.4, U1202.5, U1202.6; no longer C1205.1, U1201.4, U1201.5, U1201.6
- net 3V3: now also C1003.1, C1005.1, C1006.1, C85.1, C86.1, C87.1, C88.1, C89.1, C90.1, C91.1, C92.1, C93.1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; no longer C101.1, C102.1, C103.1, C104.1, C105.1, C106.1, C107.1, C108.1, C109.1, C1101.1, C1102.1, C1103.1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
- net 3V3_PGOOD: now also TP6.TP
- net 3V5_VIN_REG_DRVCC: now also C1227.1, R1221.2, R1222.2, R1223.2, U1202.20, U1202.24; no longer C1218.1, R1211.2, U1201.20, U1201.24
- net 5V0: now also C10.1, C1223.1, C1225.1, C1228.1, R1218.2, R1219.2, R1220.2, R1307.2, U1.1, U1202.2, U1202.21; no longer C1216.1, C1219.1, C1221.1, D1205.A, R1206.2, R1207.2, U1201.2
- net 5V0_BOOST: now also C1219.2, U1202.40; no longer C1212.2, U1201.40
- net 5V0_PGOOD: now also R1218.1, TP1.TP, U1202.23, U1202.33; no longer R1207.1, U1201.23, U1201.33, U1304.18, U1304.9, U1306.2, U1307.18, U1307.9
- net 5V0_SW: now also C1219.1, U1202.36, U1202.37, U1202.41; no longer C1212.1, U1201.36, U1201.37, U1201.41
- net AUDIO_I2C_SCL: now also R104.1; no longer R112.1
- net AUDIO_I2C_SDA: now also R103.1; no longer R110.1
- net CLK_MNGR_CLK0: now also R1005.2; no longer R1105.2
- net CLK_MNGR_CLK2: now also R1006.2; no longer R1106.2
- net CLK_MNGR_CLK4: now also R1007.2; no longer R1107.2
- net CLK_MNGR_CLKIN_SEL: now also R1001.2, U1001.6; no longer R1101.2, U1101.6
- net CLK_MNGR_REF_ACC: now also C1008.2; no longer C1108.2
- net CLK_MNGR_REF_DCC: now also C1007.1, C1008.1, R1003.2; no longer C1107.1, C1108.1, R1103.2
- net GND: now also C1.2, C10.2, C100.2, C1005.2, C1006.2, C11.2, C116.2, C117.2, C118.2, C119.2, C12.2, C120.2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; no longer C1008.2, C1009.2, C1010.2, C1104.2, C1105.2, C1106.2, C1107.2, C1219.2, C1220.2, C302.2, C303.2, C304.2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
- net N$12: now also U1001.1; no longer U1101.1
- net N$148: now also D1204.A, R1220.1; no longer D1202.A, R1206.1
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Routing:
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- removed copper zone on layer 1, net 5V0
- removed copper zone on layer 1, net 5V0_REG_VIN
- removed copper zone on layer 15, net 5V0_REG_VIN
- removed copper zone on layer 1, net 5V0_REG_VIN1
- removed copper zone on layer 1, net 5V0_SW
- removed copper zone on layer 1, net VIN

Commit message: Work on Schematic and PCB
Signed-off-by: João Silva <jgc3silva@gmail.com>
Parts:
- removed C1, C1301, C1302, C1303, C1304, C1309, C1315, C1324, C1329, C1336, C1346, C15, C2, C909, C910, C911, C912: 100nF, Capacitor:CAP0402
- removed C1305, C1325: 4.7uF, Capacitor:CAP0603
- removed C1306, C1307, C1308: 10nF, Capacitor:CAP0402
- removed C1310, C1326, C1338, C1347: 100uF, Capacitor:CAP1206
- removed C1311, C1322: 470pF, Capacitor:CAP0402
- removed C1312, C1313, C1316, C1318, C1320, C1323, C624: 10uF, Capacitor:CAP0603
- removed C1328, C913: 1uF, Capacitor:CAP0402
- removed C5, C6: 220pF, Capacitor:CAP0402
- removed C58, C97: 470nF, Capacitor:CAP0402
- removed C625, C626, C627, C628: 1nF, Capacitor:CAP0402
- removed C73: 4.7uF, Capacitor:CAP0402
- removed CON1201: 2EDG-2P-5MM, Generic Connector:2EDG-2P-5MM
- removed D1201, D1202, D1203: B0530W, Generic Diode:SOD-123
- removed F1201: 2.6A Hold, Fuses:1206
- removed L1301, L1302, L1304, L1305: 2.2uH, Coilcraft:XGL351X
- removed Q1201, Q1203, Q1205: AO4805, Alpha Omega:SOIC8
- removed Q1202, Q1204, Q1206: AO3400, Alpha Omega:SOT23
- removed R1, R1301, R1304, R1308, R1313, R1316: 10K Ohms, Resistor:RES0402
- removed R1217: 1K Ohms, Resistor:RES0402
- removed R1302: 301K Ohms, Resistor:RES0402
- removed R1303: 158K Ohms, Resistor:RES0402
- removed R1305: 118K Ohms, Resistor:RES0402
- removed R1306: 100K Ohms, Resistor:RES0402
- removed R1307: 10K Ohms, Resistor:RES0603
- removed R1309: 324K Ohms, Resistor:RES0402
- removed R1310: 107K Ohms, Resistor:RES0402
- removed R1311: 274K Ohms, Resistor:RES0603
- removed R1312: 294K Ohms, Resistor:RES0603
- removed R1314: 309K Ohms, Resistor:RES0402
- removed R1315: 71.5K Ohms, Resistor:RES0402
- removed R2: TBD Ohms, Resistor:RES0402
- removed R804, R806: 2.21K Ohms, Resistor:RES0402
- removed R805: 49.9K Ohms, Resistor:RES0402
- removed RFCON701, RFCON702: RFCON-SMA, RF Connector:SMA
- removed U1, U602, U603: MIC2019, Microchip:SOT23-6
- removed U1301: ADM7172ACPZ-5.0, Analog Devices:LFCSP8_3X3
- removed U1302, U1303: ADM7171ACPZ-1.3, Analog Devices:LFCSP8_3X3
- removed U1307: MIC23159, Microchip:VQFN20
- removed U1308: ADP7142AUJZ-3.3, Analog Devices:SOT23-5
- removed U801: ADAU1372, Analog Devices:QFN40
- added C1104: 1uF, Capacitor:CAP0603
- added C1105, C1110, C1111, C1112: 10uF, Capacitor:CAP1206
- added C1106, C1107, C1109, C1113, C1120, C1121, C1129, C1130, C1243, C1252, C347, C348, C349, C350, C405, C421, C426, C707, C709, C710, C711, C712: 100nF, Capacitor:CAP0402
- added C1108, C1115, C224, C229, C351: 4.7uF, Capacitor:CAP0402
- added C1114, C1126, C1235, C1239, C410, C708: 10uF, Capacitor:CAP0603
- added C1116, C1117, C1118, C1119, C1127, C1128: 4.7uF, Capacitor:CAP0603
- added C1122, C1123, C1124, C1125, C1244, C1253: 100uF, Capacitor:CAP1206
- added C1231, C406, C407, C411, C412, C416, C417, C418, C419: 10nF, Capacitor:CAP0402
- added C234, C239: 470nF, Capacitor:CAP0402
- added C262, C269, C352, C713: 47uF, Capacitor:CAP0603
- added C408, C409, C413, C414, C415, C420, C422, C424: 1uF, Capacitor:CAP0402
- added C423, C425: 1nF, Capacitor:CAP0402
- added C427: DNP, Capacitor:CAP0402
- added C428: 10pF, Capacitor:CAP0402
- added CON1101: 2EDG-2P-5MM-H, Generic Connector:2EDG-2P-5MM-H
- added D1001, D1101, D1102, D1103: B0530W, Generic Diode:SOD-123
- added D101: LED0603, LED:0603
- added D201: RGBLED, LED:5050
- added F1001: (no value), PTC Fuses:1206
- added FB601: 1uH, Inductor:IND0603
- added L1001: 0603USB-951ML, Coilcraft:0603USB
- added L1102: 2.2uH, Coilcraft:XGL6030
- added L1203, L1204: 2.2uH, Coilcraft:XGL351X
- added L501, L502: 330nH, Inductor:IND0805
- added Q101, Q1102, Q1103, Q1106: AO3400, Alpha Omega:SOT23
- added Q1101, Q1104, Q1105: AO4805, Alpha Omega:SOIC8
- added R106, R109, R1124, R1125: DNP, Resistor:RES0402
- added R110, R1106, R1107, R1113, R1114, R1116, R1117, R505, R506, R511, R512: 1K Ohms, Resistor:RES0402
- added R1105, R1112, R1115, R1118, R509, R510: 10K Ohms, Resistor:RES0402
- added R1108, R1110, R904: 100K Ohms, Resistor:RES0402
- added R1109, R1111: 5.1K Ohms, Resistor:RES0402
- added R111, R112: 220 Ohms, Resistor:RES0402
- added R113, R114: 2.2K Ohms, Resistor:RES0402
- added R206: 4.7K Ohms, Resistor:RES0402
- added R207: 330 Ohms, Resistor:RES0402
- added R305, R306, R307, R308: 40.2 Ohms, Resistor:RES0402
- added R507, R508: TBD Ohms, Resistor:RES0402
- added R513: 49.9 Ohms, Resistor:RES0402
- added R514: 10 Ohms, Resistor:RES0402
- added R905, R906, R907, R908, R909, R910, R911, R912: 0 Ohms, Resistor:RES0402
- added RFCON401: RFCON-U.FL, RF Connector:U.FL
- added RFCON502: RFCON-SMA-RA, RF Connector:SMA-RA
- added TP10, TP11, TP12, TP13, TP14, TP8, TP9: TESTPOINT-0.7MM, PADs:PAD0.7MM
- added U101: MIC2019, Microchip:SOT23-6
- added U1102: LT7182S, Analog Devices:LQFN40_ASYM_CORNER
- added U1203, U1207: ADM7171ACPZ-3.3, Analog Devices:LFCSP8_3X3
- added U1206: ADM7171ACPZ-1.3, Analog Devices:LFCSP8_3X3
- added U1208: MIC23159, Microchip:VQFN20
- added U1210: ADP7142AUJZ-3.3, Analog Devices:SOT23-5
- added U302: MT41K256M16TW-125, Micron:FBGA96_14X8
- added U303: DSC1203DA3-333M3333, Microchip:VDFN6
- added U901: 74LVC1G157, Logic:SC70-6
- added U902: DSB321SDA, Crystal:TCXO-3225
- added U903: SI5351C-B-GM, Silicon Labs:QFN20
- C1002, C1003: value 100nF -> 220pF
- C1007, C1008: value 10pF -> 100nF
- C101, C1224: value 4.7uF -> 100nF
- C102, C1214: value 4.7uF -> 10uF; device Capacitor:CAP0402 -> Capacitor:CAP0603
- C103, C301: value 470nF -> 100nF
- C104: value 470nF -> 1uF
- C1103: value 100nF -> 10uF; device Capacitor:CAP0402 -> Capacitor:CAP1206
- C1203: value 10uF -> 100nF; device Capacitor:CAP1206 -> Capacitor:CAP0402
- C1204, C1228: value 1uF -> 100nF; device Capacitor:CAP0603 -> Capacitor:CAP0402
- C1205: value 10uF -> 4.7uF; device Capacitor:CAP1206 -> Capacitor:CAP0603
- C1206, C1207, C402: value 100nF -> 10nF
- C1208: value 4.7uF -> 10nF; device Capacitor:CAP0603 -> Capacitor:CAP0402
- C1210: value 10uF -> 100uF
- C1211: value 10uF -> 470pF; device Capacitor:CAP1206 -> Capacitor:CAP0402
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- renumbered C10 to C1013, C100 to C219, C105 to C244, C106 to C249, C107 to C254, C108 to C259, C109 to C205, C11 to C309, C110 to C210, C111 to C215, C112 to C220, C113 to C225, C114 to C230, C115 to C235, C116 to C240, C117 to C245, C118 to C250, C119 to C255, C12 to C314, C120 to C260, C121 to C263, C122 to C267, C123 to C270, C124 to C264, C125 to C268, C126 to C271, C13 to C323, C1314 to C1234, C1317 to C1238, C1319 to C1241, C1321 to C1242, C1327 to C1245, C1330 to C1246, C1331 to C1230, C1332 to C1232, C1333 to C1237, C1334 to C1250, C1335 to C1240, C1337 to C1233, C1339 to C1236, C1340 to C1247, C1341 to C1257, C1342 to C1259, C1343 to C1248, C1344 to C1249, C1345 to C1251, C1348 to C1254, C1349 to C1256, C1350 to C1255, C1351 to C1258, C14 to C328, C16 to C305, C17 to C310, C18 to C315, C19 to C319, C20 to C324, C21 to C329, C22 to C334, C23 to C339, C24 to C302, C25 to C306, C26 to C311, C27 to C316, C28 to C320, C29 to C325, C3 to C1010, C30 to C330, C31 to C335, C32 to C340, C33 to C303, C34 to C307, C35 to C312, C36 to C317, C37 to C321, C38 to C326, C39 to C331, C4 to C1012, C40 to C336, C41 to C341, C42 to C304, C43 to C308, C44 to C313, C45 to C318, C46 to C322, C47 to C327, C48 to C332, C49 to C337, C50 to C342, C51 to C344, C52 to C345, C53 to C333, C54 to C338, C55 to C343, C56 to C346, C60 to C206, C61 to C211, C62 to C216, C629 to C529, C63 to C221, C630 to C530, C631 to C531, C632 to C532, C633 to C533, C634 to C534, C635 to C535, C636 to C536, C637 to C537, C638 to C538, C639 to C539, C64 to C226, C640 to C540, C641 to C541, C642 to C542, C643 to C543, C644 to C544, C645 to C545, C646 to C546, C647 to C547, C648 to C548, C649 to C549, C65 to C231, C650 to C550, C651 to C551, C652 to C552, C653 to C553, C654 to C554, C66 to C236, C67 to C241, C68 to C246, C69 to C251, C7 to C1009, C70 to C256, C71 to C261, C72 to C265, C74 to C207, C75 to C212, C76 to C217, C77 to C222, C78 to C227, C79 to C232, C8 to C1011, C80 to C237, C81 to C242, C814 to C714, C815 to C715, C816 to C716, C817 to C717, C818 to C718, C819 to C719, C82 to C247, C820 to C720, C821 to C721, C822 to C722, C83 to C252, C84 to C257, C85 to C266, C86 to C208, C87 to C213, C88 to C218, C89 to C223, C9 to C1014, C90 to C228, C91 to C233, C92 to C238, C93 to C243, C94 to C248, C95 to C253, C96 to C258, C98 to C209, C99 to C214, CON201 to CON101, CON901 to CON801, D1204 to D1104, D1205 to D1105, D601 to D501, D602 to D502, D603 to D503, D604 to D504, FB501 to FB401, FB502 to FB402, FB801 to FB701, J201 to J101, J801 to J701, J802 to J702, J803 to J703, L1303 to L1205, L603 to L503, L604 to L504, L605 to L505, L606 to L506, L607 to L507, L608 to L508, L609 to L509, L610 to L510, L611 to L511, L612 to L512, L801 to L701, L802 to L702, M801 to M701, M802 to M702, R1218 to R1119, R1219 to R1120, R1220 to R1121, R1221 to R1122, R1222 to R1123, R1223 to R1126, R1224 to R1127, R1225 to R1128, R1226 to R1129, R1227 to R1130, R3 to R302, R4 to R209, R405 to R309, R406 to R310, R407 to R311, R408 to R312, R409 to R301, R410 to R313, R411 to R314, R412 to R315, R413 to R316, R414 to R317, R415 to R318, R416 to R319, R417 to R320, R418 to R321, R419 to R322, R420 to R323, R421 to R324, R422 to R325, R423 to R326, R424 to R327, R425 to R328, R426 to R329, R427 to R330, R428 to R304, R429 to R303, R5 to R210, R6 to R208, R615 to R515, R616 to R516, R807 to R707, R808 to R708, R809 to R709, R810 to R710, R811 to R711, RFCON1001 to RFCON901, RFCON1002 to RFCON902, RFCON603 to RFCON503, RFCON604 to RFCON504, RFCON605 to RFCON505, RFCON606 to RFCON506, RFCON607 to RFCON507, RFCON608 to RFCON508, RFCON609 to RFCON509, RFCON610 to RFCON510, SD201 to SD101, SHIELD501 to SHIELD401, T601 to T501, T602 to T502, T603 to T503, T604 to T504, T605 to T505, T606 to T506, T607 to T507, T608 to T508, TC1101 to TC1001, TC301 to TC201, U1304 to U1204, U1305 to U1205, U1306 to U1209, U1309 to U1211, U202 to U102, U604 to U504, U605 to U505, U606 to U506, USB1101 to USB1001
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Connections:
- removed net N$92: C1204.1, D1201.C, D1202.C, D1203.C, U1201.1, U1201.4
- removed net SMC_MAIN_CLK: R1012.1
- removed net VDD: U403.6
- new net !CM4_ACT_LED: D101.C, U102.21
- new net !CM4_BTLDR: U102.93
- new net !CM4_PWR_LED: Q101.1, U102.95
- new net !SYNTH_RESET: R601.2, U601.31
- new net !SYNTH_SPI_CS: U601.25
- new net !VBUS_SRC_FAULT: R1010.1, U1003.4
- new net !VIN_REG_ALERT: R1118.1, U1102.29
- new net 3V3_SYNTH_IN_PD_FB: C1214.1, C1217.1, C603.1, C606.1, C609.1, FB601.1, R603.2, R605.2, U1203.1, U1203.2, U1203.3, U601.12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
- new net 3V3_SYNTH_VCO_RF: C1235.1, C1239.1, C602.1, C604.1, C607.1, C610.1, L601.1, L602.1, U1207.1, U1207.2, U1207.3, U601.3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
- new net CM4_GLOBAL_EN: R101.2, U102.99
- new net CM4_PTP_PPS: R108.2, R109.2
- new net CM4_RUNNING: U102.92
- new net CM4_USB_OTG: U102.101
- new net FPGA_CLK0: R905.1, U201.W11
- new net FPGA_CLK1: R909.1, U201.V13
- new net FPGA_CLK2: R906.1, U201.W19
- new net FPGA_CLK3: R910.1, U201.Y18
- new net N$100: C621.2, R614.2
- new net N$101: C615.1, R607.1
- new net N$102: C620.2, R613.2
- new net N$103: C618.1, L601.2, R609.2, R611.2
- new net N$104: C620.1, R611.1, U601.39
- new net N$105: C617.1, R608.1, U601.5
- new net N$106: C622.1, R609.1, U601.40
- new net N$107: C621.1, R612.1, U601.46
- new net N$108: C623.1, R610.1, U601.45
- new net N$109: C616.1, R607.2, R608.2, U601.10
- new net N$110: R1007.1, U1002.25
- new net N$111: R1007.2, TP11.TP, U1002.20
- new net N$112: TP8.TP, U1002.24
- new net N$113: TP10.TP, U1002.23
- new net N$114: TP9.TP, U1002.22
- new net N$115: TP12.TP, U1002.29
- new net N$116: R108.1, U102.18
- new net N$117: R109.1, U102.16
- new net N$118: R105.2, U102.91
- new net N$119: R104.2, U102.89
- new net N$120: R106.2, U102.20
- new net N$121: D101.A, R107.1
- new net N$122: TP13.TP, U102.111
- new net N$123: D102.A, Q101.3, R110.1
- new net N$124: R1124.1, U1102.26
- new net N$125: R1125.1, U1102.24
- new net N$96: C1208.1, U1203.4
- new net N$97: C1231.1, U1207.4
- new net N$98: C614.1, FB601.2, U601.18
- new net N$99: C623.2, RFCON602.SIGNAL
- new net PM_I2C_EN: R1002.2, U1001.1
- new net PM_I2C_SCL: R1003.1, U1001.2, U1002.32, U1102.30
- new net PM_I2C_SDA: R1004.1, U1001.7, U1002.31, U1102.31
- new net SYNTH_CE: R602.2, U601.29
- new net SYNTH_LD: U601.8
- new net SYNTH_MUTE: U601.7
- new net SYNTH_SPI_MISO: U601.27
- new net SYNTH_SPI_MOSI: U601.28
- new net SYNTH_SPI_SCK: U601.26
- new net VIN_PM: C1104.1, D1101.C, D1102.C, D1103.C, U1101.1, U1101.4
- net !1V0_FAULT: now also U1102.27; no longer U1202.27
- net !5V0_FAULT: now also U1102.28; no longer U1202.28
- net !5V0_TRX_BIAS_T1_OC: now also R503.1, U501.4; no longer R603.1, U601.4
- net !5V0_TRX_BIAS_T2_OC: now also R504.1, U502.4; no longer R604.1, U602.4
- net !5V0_TRX_PA1_OC: now also R509.1, U503.4; no longer R609.1, U603.4
- net !5V0_TRX_PA2_OC: now also R510.1; no longer R610.1
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Routing:
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Other:
- board text added: "IcyRadio v2 Sep 2022"
- board text removed: "IcyRadio v2 Jun 2021"
