File: pcb/main/icyradio-main.brd (EAGLE design)
At the start: 167.7 x 111.2 mm, 689 parts, among them CON101 FPC-22P, CON1101 2EDG-2P-5MM-H, CON801 PCIE-X4-EDGE, J101 RJ45_MAG_LED_1G-TE-1-2301994-0, J701 TRSJACK, J702 TRSJACK, J703 TRSJACK, M701 SPH0641LM4H-1, M702 SPH0641LM4H-1, Q101 AO3400, Q1101 AO4805, Q1102 AO3400, Q1103 AO3400, Q1104 AO4805, Q1105 AO4805, Q1106 AO3400, T501 UWB1-85E, T502 UWB1-85E, T503 UWB1-85E, T504 UWB1-85E, T505 UWB1-85E, T506 UWB1-85E, T507 UWB1-85E, T508 UWB1-85E, U1001 LTC4313-3, U1002 UPD301C, U1003 MIC2019, U101 MIC2019, U102 RPI-CM4, U1101 MCP1804-3302, U1102 LT7182S, U1201 ADM7172ACPZ-5.0, U1202 ADM7171ACPZ-1.3, U1203 ADM7171ACPZ-3.3, U1204 MIC23159, U1205 MIC5166, U1206 ADM7171ACPZ-1.3, U1207 ADM7171ACPZ-3.3, U1208 MIC23159, U1209 MIC23155, U1210 ADP7142AUJZ-3.3, U1211 ADP150UJZ-1.8, U201 XC7A100TFGG484, U301 MT41K256M16TW-125, U302 MT41K256M16TW-125, U303 DSC1203DA3-333M3333, U401 AD9361, U402 LTC6957-3, U403 TG2520SMN-40.0000M, U501 MIC2019, U502 MIC2019, U503 MIC2019, U504 MIC2019, U505 ADL5601, U506 ADL5601, U601 8V97003, U701 ADAU1372, U901 74LVC1G157, U902 DSB321SDA, U903 SI5351C-B-GM

Commit message: PCB Work
Signed-off-by: João Silva <jgc3silva@gmail.com>
Parts:
- removed R1122, R1123: 10K Ohms, Resistor:RES0402
- added C1: 100nF, Capacitor:CAP0402
- added D2, D3, D4: LED0603, LED:0603
- added R1: 22 Ohms, Resistor:RES0402
- added R10, R8, R9: 1K Ohms, Resistor:RES0402
- added R2: 2.4K Ohms, Resistor:RES0402
- added R3, R4, R5, R6, R7: 4.7K Ohms, Resistor:RES0402
- added U1: SST26VF064B, Microchip:WSOIC8
- C102, C1114, C1126, C1128, C1213, C1214, C1216, C1217, C1218, C1219, C1220, C1222, C1233, C1234, C1235, C1236, C1238, C1239, C1241, C1242, C1254, C1255, C410, C534, C535, C605, C608, C611, C612, C613, C701, C706, C708, C721, C722: device Capacitor:CAP0603 -> Capacitor:CAP0402
- C1259: value 4.7uF -> 10uF; device Capacitor:CAP0603 -> Capacitor:CAP0402
- R1210, R1215, R1216, R401: device Resistor:RES0603 -> Resistor:RES0402
- moved C1002 887.1 mm to (-247.5, 10.5)
- moved C1003 887.1 mm to (-247.5, 13.0)
- moved C1007 887.1 mm to (-247.5, 23.0)
- moved C1008 887.1 mm to (-247.5, 20.5)
- moved C1009 887.1 mm to (-247.5, 0.50)
- moved C1010 887.1 mm to (-247.5, 18.0)
- moved C1011 887.1 mm to (-247.5, -2.00)
- moved C1012 887.1 mm to (-247.5, 15.5)
- moved C1013 887.1 mm to (-247.5, -12.0)
- moved C1014 887.1 mm to (-247.5, -4.50)
- moved C1102 887.1 mm to (-247.5, 92.5)
- moved C1107 887.1 mm to (-244.0, 92.5)
- moved C201 887.1 mm to (-247.5, -108.0)
- moved C301 887.1 mm to (-247.5, -28.0)
- moved C302 887.1 mm to (-247.5, -55.5)
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Connections:
- net N$124 renamed VIN_REG_WP
- net N$125 renamed VIN_REG_RUN0
- net N$19 renamed VIN_REG_ASEL
- removed net !1V0_FAULT: R1123.1, U1102.27
- removed net !5V0_FAULT: R1122.1, U1102.28
- new net !FPGA_FLASH_CS: R2.1, U1.1, U201.T19
- new net !FPGA_INIT: D4.A, R10.1, R6.1, U201.U12
- new net !FPGA_PROGRAM: R7.1, TC201.9, U201.N12
- new net FPGA_DONE: D3.A, R9.1, U201.G11
- new net FPGA_FLASH_IO0: U1.5, U201.P22
- new net FPGA_FLASH_IO1: U1.2, U201.R22
- new net FPGA_FLASH_IO2: R3.1, U1.3, U201.P21
- new net FPGA_FLASH_IO3: R4.1, U1.7, U201.R21
- new net FPGA_FLASH_SCK: U1.6, U201.L12, U201.N13
- new net FPGA_JTAG_EN: R5.2, TC201.10, U201.U9
- new net N$19: D2.A, R8.1
- new net TRX_SYNC_IN: R1.2, U201.F18, U401.H5
- net 2V5: now also U201.D15, U201.D16, U201.F20, U201.F21
- net 3V3: now also C1.1, R10.2, R2.2, R3.2, R4.2, R6.2, R7.2, R9.2, U1.8, U201.U11
- net 3V5_VIN_REG_DRVCC: now also U1102.27, U1102.28; no longer R1122.2, R1123.2
- net GND: now also C1.2, D2.C, D3.C, D4.C, R5.1, U1.4, U201.H19, U201.H20, U201.M20, U201.M21, U201.N10, U201.N9, U201.U10, U201.U22; no longer U401.H5
- net TRX_CTRL_OUT3: now also U201.D17; no longer U201.E18
- net TRX_ENABLE: now also U201.F16; no longer U201.F18
- net TRX_EN_AGC: now also U201.F15; no longer U201.F16
- net TRX_TX/!RX: now also U201.F14; no longer U201.F15
- net VBUS: now also Q1101.5, Q1101.6; no longer Q1101.7, Q1101.8
- net VIN: now also Q1101.7, Q1101.8; no longer Q1101.5, Q1101.6
Routing:
- net GND: track 107.1 -> 177.0 mm, vias 74 -> 110
- net TRX_SYNC_IN: track 0.00 -> 33.7 mm, vias 0 -> 2
- net 1V0: track 0.00 -> 26.9 mm, vias 0 -> 21
- net 2V5: track 0.00 -> 15.0 mm, vias 0 -> 11
- net 1V35: track 0.00 -> 8.47 mm, vias 0 -> 12
- net 1V8: track 0.00 -> 5.66 mm, vias 0 -> 7
- net 1V2: track 0.00 -> 4.95 mm, vias 0 -> 4
- net 3V3: track 1.10 -> 5.34 mm, vias 1 -> 6
- net TRX_ENABLE: track 35.4 -> 38.4 mm
- net 0V675_DDR3_VREF: track 0.00 -> 2.83 mm, vias 0 -> 4
- net FPGA_FLASH_SCK: track 0.00 -> 1.41 mm, vias 0 -> 2
- net TRX_EN_AGC: track 38.8 -> 39.8 mm
- net TRX_TX/!RX: track 38.9 -> 39.9 mm
- net TRX_CTRL_IN3: track 28.7 -> 29.7 mm
- net TRX_CTRL_IN2: track 26.8 -> 27.8 mm
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- added copper zone on layer 1, net 1V2_SW
- added copper zone on layer 1, net 1V35
- added copper zone on layer 1, net 1V35_SW
- added copper zone on layer 1, net 1V8
- added copper zone on layer 1, net 1V8_SW

Commit message: PCB Work
Signed-off-by: João Silva <jgc3silva@gmail.com>
Parts:
- added C2: 1uF, Capacitor:CAP0402
- added CON1: FPC-22P, Generic Connector:FPC-22P
- added R11, R12: 2.2K Ohms, Resistor:RES0402
- moved D4 511.6 mm to (35.7, 119.2), turned to 270 degrees
- moved R10 511.4 mm to (37.8, 119.4), turned to 270 degrees
- moved R9 510.9 mm to (39.9, 119.4), turned to 270 degrees
- moved D3 510.2 mm to (42.0, 119.2), turned to 270 degrees
- moved R8 510.0 mm to (44.1, 119.4), turned to 270 degrees
- moved D2 509.3 mm to (46.2, 119.2), turned to 270 degrees
- moved R7 509.1 mm to (48.3, 119.4), turned to 270 degrees
- moved R6 508.7 mm to (50.4, 119.4), turned to 270 degrees
- moved R1 508.4 mm to (75.2, 120.3), turned to 270 degrees
- moved R5 508.3 mm to (52.5, 119.4), turned to 270 degrees
- moved R4 465.0 mm to (55.1, 62.8), turned to 90 degrees
- moved R3 462.8 mm to (54.1, 62.8), turned to 90 degrees
- moved R2 462.6 mm to (56.1, 62.8), turned to 90 degrees
- moved C1 461.8 mm to (57.1, 62.8), turned to 270 degrees
- moved U1 456.5 mm to (60.9, 60.9)
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Connections:
- net CM4_CAM_SCL renamed CM4_CAM1_SCL
- net CM4_CAM_SDA renamed CM4_CAM1_SDA
- net N$100 renamed SYNTH_RFOUTB_ACC_N
- net N$102 renamed SYNTH_RFOUTA_ACC_N
- net N$103 renamed SYNTH_RFOUTA_BIAS
- net N$104 renamed SYNTH_RFOUTA_N
- net N$105 renamed SYNTH_VTUNE
- net N$106 renamed SYNTH_RFOUTA_P
- net N$107 renamed SYNTH_RFOUTB_N
- net N$108 renamed SYNTH_RFOUTB_P
- net N$109 renamed SYNTH_CPOUT
- net N$33 renamed PCIE_SLOT_TX1_ACC_N
- net N$34 renamed PCIE_SLOT_TX1_ACC_P
- net N$35 renamed PCIE_SLOT_RX1_ACC_N
- net N$41 renamed PCIE_SLOT_RX1_ACC_P
- net N$43 renamed SYNTH_CPBIAS
- net N$45 renamed PCIE_SLOT_RX0_ACC_N
- net N$46 renamed PCIE_SLOT_RX0_ACC_P
- net N$51 renamed PCIE_CM4_RX_ACC_N
- net N$53 renamed PCIE_CM4_RX_ACC_P
- net N$63 renamed PCIE_SLOT_TX0_ACC_N
- net N$65 renamed PCIE_SLOT_TX0_ACC_P
- net N$68 renamed PCIE_CM4_TX_ACC_N
- net N$69 renamed PCIE_CM4_TX_ACC_P
- net N$75 renamed SYNTH_VREGVCO1
- net N$76 renamed SYNTH_VREGVCO2
- net N$77 renamed SYNTH_VREFVCO1
- net N$84 renamed SYNTH_VREFVCO2
- net N$85 renamed SYNTH_RFOUTB_BIAS
- net N$86 renamed SYNTH_RFOUTA_ACC_P
- net N$88 renamed SYNTH_REFIN_P
- net N$89 renamed SYNTH_REFIN_N
- net N$99 renamed SYNTH_RFOUTB_ACC_P
- new net CM4_CAM0_CSI_C_N: CON1.15, U102.140
- new net CM4_CAM0_CSI_C_P: CON1.14, U102.142
- new net CM4_CAM0_CSI_D0_N: CON1.21, U102.128
- new net CM4_CAM0_CSI_D0_P: CON1.20, U102.130
- new net CM4_CAM0_CSI_D1_N: CON1.18, U102.134
- new net CM4_CAM0_CSI_D1_P: CON1.17, U102.136
- new net CM4_CAM0_SCL: CON1.3, R12.1, U102.35
- new net CM4_CAM0_SDA: CON1.2, R11.1, U102.36
- net 3V3_CM4: now also C2.1, CON1.1, R11.2, R12.2
- net CM4_CAM_GPIO: now also CON1.6
- net GND: now also C2.2, CON1.10, CON1.13, CON1.16, CON1.19, CON1.22, CON1.4, CON1.7
- net TRX_DATA_CLK: now also U201.K18; no longer U201.J19
- net TRX_FB_CLK: now also U201.J19; no longer U201.K18
Routing:
- net FPGA_FLASH_SCK: track 1.41 -> 42.6 mm, vias 2 -> 3
- net FPGA_FLASH_IO2: track 0.71 -> 39.1 mm, vias 1 -> 5
- net FPGA_FLASH_IO0: track 0.71 -> 33.7 mm, vias 1 -> 4
- net GND: track 177.0 -> 208.7 mm, vias 110 -> 127
- net FPGA_FLASH_IO3: track 0.71 -> 30.4 mm, vias 1 -> 3
- net FPGA_FLASH_IO1: track 0.70 -> 27.2 mm, vias 1 -> 3
- net !FPGA_FLASH_CS: track 0.71 -> 26.6 mm, vias 1 -> 3
- net 3V3: track 5.34 -> 11.0 mm, vias 6 -> 14
- net 2V5_TRX_INTERFACE: track 1.50 -> 2.97 mm, vias 0 -> 1
- net TRX_FB_CLK: track 23.8 -> 22.5 mm
- net TRX_DATA_CLK: track 21.7 -> 22.7 mm
- net 1V8: track 5.66 -> 6.36 mm, vias 7 -> 8
- net 1V3_TRX: track 3.56 -> 2.95 mm, vias 2 -> 3
- added copper zone on layer 14, net GND
- added copper zone on layer 3, net GND
- added copper zone on layer 3, net N$124
- added copper zone on layer 14, net N$92

Commit message: PCB Work
Signed-off-by: João Silva <jgc3silva@gmail.com>
Parts:
- added C3: 1uF, Capacitor:CAP0402
- added C4: 100nF, Capacitor:CAP0402
- added FB1: 1uH, Inductor:IND0603
- added R13: 49.9 Ohms, Resistor:RES0402
- R902, R904: value 100K Ohms -> 10K Ohms
Connections:
- new net N$34: C902.1, C904.1, C905.1, FB1.2, U903.10, U903.11, U903.14, U903.18
- new net SYNTH_REF_CLK: C601.1, R13.2
- net 3V3: now also C3.1, FB1.1; no longer C902.1, C904.1, C905.1, U903.10, U903.11, U903.14, U903.18
- net EXT_CLK_OUT: now also R912.1; no longer R911.1
- net GND: now also C3.2, C4.2, R13.1
- net SYNTH_REFIN_N: now also C4.1

Commit message: Start DDR routing
Signed-off-by: João Silva <jgc3silva@gmail.com>
Parts:
- removed U1211: ADP150UJZ-1.8, Analog Devices:SOT23-5
- added U2: ADP7142AUJZ-1.8, Analog Devices:SOT23-5
- moved C1245 103.5 mm to (125.3, 64.3)
- moved C1250 103.5 mm to (126.3, 64.3)
- moved C1246 103.5 mm to (124.1, 64.8)
- moved C1257 103.5 mm to (121.9, 64.8)
- moved C1259 103.5 mm to (121.9, 63.8)
- moved L1205 103.5 mm to (120.4, 61.3)
- moved R1210 103.5 mm to (125.9, 58.3)
- moved R1215 103.5 mm to (123.9, 58.3)
- moved R1216 103.5 mm to (124.9, 58.3)
- moved U1209 103.5 mm to (124.4, 61.3)
- moved C1209 97.2 mm to (106.1, 68.4)
- moved C1201 97.2 mm to (113.8, 70.3)
- moved C1205 97.2 mm to (115.8, 70.2)
- moved C1210 97.2 mm to (107.5, 63.0)
- moved C1211 97.2 mm to (109.8, 74.8)
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Connections:
- new net CM4_UART_RXD: U102.51
- new net CM4_UART_TXD: U102.55
- new net CM4_WAKE: U102.56
- net 1V8_TRX_REF: now also U2.4, U2.5; no longer U1211.5
- net 2V5: now also U2.1; no longer U1211.1
- net GND: now also U2.2; no longer U1211.2
- net TRX_REF_EN: now also U2.3; no longer U1211.3
Routing:
- net DDR3_A6: track 0.00 -> 45.5 mm, vias 0 -> 4
- net DDR3_A5: track 0.00 -> 45.4 mm, vias 0 -> 3
- net DDR3_A0: track 0.00 -> 45.2 mm, vias 0 -> 4
- net DDR3_A4: track 0.00 -> 44.8 mm, vias 0 -> 4
- net DDR3_ODT: track 0.00 -> 44.7 mm, vias 0 -> 5
- net DDR3_BA0: track 0.00 -> 44.7 mm, vias 0 -> 4
- net DDR3_A9: track 0.00 -> 44.5 mm, vias 0 -> 3
- net DDR3_A1: track 0.00 -> 44.5 mm, vias 0 -> 4
- net !DDR3_WE: track 0.00 -> 44.4 mm, vias 0 -> 6
- net DDR3_A13: track 0.00 -> 44.3 mm, vias 0 -> 3
- net !DDR3_CS: track 0.00 -> 44.3 mm, vias 0 -> 5
- net DDR3_BA1: track 0.00 -> 44.1 mm, vias 0 -> 3
- net DDR3_A2: track 0.00 -> 44.1 mm, vias 0 -> 4
- net DDR3_A10: track 0.00 -> 44.0 mm, vias 0 -> 3
- net DDR3_A7: track 0.00 -> 43.9 mm, vias 0 -> 3
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