File: pcb/main/icyradio-main.sch (EAGLE design)
At the start: 707 parts, among them CON1 FPC-22P, CON101 FPC-22P, CON1101 2EDG-2P-5MM-H, CON801 PCIE-X4-EDGE, J101 RJ45_MAG_LED_1G-TE-1-2301994-0, J701 TRSJACK, J702 TRSJACK, J703 TRSJACK, M701 SPH0641LM4H-1, M702 SPH0641LM4H-1, Q101 AO3400, Q1101 AO4805, Q1102 AO3400, Q1103 AO3400, Q1104 AO4805, Q1105 AO4805, Q1106 AO3400, T501 UWB1-85E, T502 UWB1-85E, T503 UWB1-85E, T504 UWB1-85E, T505 UWB1-85E, T506 UWB1-85E, T507 UWB1-85E, T508 UWB1-85E, U1 SST26VF064B, U1001 LTC4313-3, U1002 UPD301C, U1003 MIC2019, U101 MIC2019, U102 RPI-CM4, U1101 MCP1804-3302, U1102 LT7182S, U1201 ADM7172ACPZ-5.0, U1202 ADM7171ACPZ-1.3, U1203 ADM7171ACPZ-3.3, U1204 MIC23159, U1205 MIC5166, U1206 ADM7171ACPZ-1.3, U1207 ADM7171ACPZ-3.3, U1208 MIC23159, U1209 MIC23155, U1210 ADP7142AUJZ-3.3, U2 ADP7142AUJZ-1.8, U201 XC7A100TFGG484, U302 MT41K256M16TW-125, U303 DSC1203DA3-333M3333, U401 AD9361, U402 LTC6957-3, U403 TG2520SMN-40.0000M, U501 MIC2019, U502 MIC2019, U503 MIC2019, U504 MIC2019, U505 ADL5601, U506 ADL5601, U601 8V97003, U701 ADAU1372, U901 74LVC1G157, U902 DSB321SDA, U903 SI5351C-B-GM

Commit message: DDR3 routing finished Some more PCB progress
Signed-off-by: João Silva <jgc3silva@gmail.com>
Other:
- note added: "0.675V"
- note removed: "0.625V"
- note removed: "TODO: - Connect IOs - Find IOs scattered around"
- moved on the sheet: R201, R202, R203, R206
Changed lines of the file:
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@@
 <description>FPGA</description>
 <plain>
-<text x="340.36" y="411.48" size="6.4516" layer="98">TODO:
-- Connect IOs
-- Find IOs scattered around</text>
 <text x="119.38" y="142.24" size="6.4516" layer="97" rot="R90" align="center">2V5</text>
 <text x="119.38" y="58.42" size="6.4516" layer="97" rot="R90" align="center">2V5</text>
@@
 <attribute name="VALUE" x="347.98" y="365.76" size="1.778" layer="96" rot="R90"/>
 </instance>
-<instance part="R206" gate="G$1" x="-76.2" y="210.82" smashed="yes" rot="R270">
-<attribute name="VALUE" x="-78.9686" y="210.82" size="1.778" layer="96" ratio="10" rot="SR270" align="top-left"/>
-<attribute name="NAME" x="-73.4314" y="210.82" size="1.778" layer="95" ratio="10" rot="SR270"/>
-<attribute name="TOLERANCE" x="-81.5086" y="210.82" size="1.778" layer="97" ratio="10" rot="SR270" align="top-left"/>
-</instance>
-<instance part="3V3116" gate="G$1" x="-76.2" y="215.9" smashed="yes">
-<attribute name="VALUE" x="-78.74" y="213.36" size="1.778" layer="96" rot="R90"/>
-</instance>
-<instance part="R203" gate="G$1" x="-88.9" y="210.82" smashed="yes" rot="R270">
-<attribute name="VALUE" x="-91.6686" y="210.82" size="1.778" layer="96" ratio="10" rot="SR270" align="top-left"/>
-<attribute name="NAME" x="-86.1314" y="210.82" size="1.778" layer="95" ratio="10" rot="SR270"/>
-<attribute name="TOLERANCE" x="-94.2086" y="210.82" size="1.778" layer="97" ratio="10" rot="SR270" align="top-left"/>
-</instance>
-<instance part="3V3115" gate="G$1" x="-88.9" y="215.9" smashed="yes">
-<attribute name="VALUE" x="-91.44" y="213.36" size="1.778" layer="96" rot="R90"/>
-</instance>
-<instance part="R202" gate="G$1" x="-111.76" y="210.82" smashed="yes" rot="R270">
-<attribute name="VALUE" x="-114.5286" y="210.82" size="1.778" layer="96" ratio="10" rot="SR270" align="top-left"/>
-<attribute name="NAME" x="-108.9914" y="210.82" size="1.778" layer="95" ratio="10" rot="SR270"/>
-<attribute name="TOLERANCE" x="-117.0686" y="210.82" size="1.778" layer="97" ratio="10" rot="SR270" align="top-left"/>
-</instance>
-<instance part="3V3113" gate="G$1" x="-111.76" y="215.9" smashed="yes">
-<attribute name="VALUE" x="-114.3" y="213.36" size="1.778" layer="96" rot="R90"/>
-</instance>
-<instance part="R201" gate="G$1" x="-124.46" y="210.82" smashed="yes" rot="R270">
-<attribute name="VALUE" x="-127.2286" y="210.82" size="1.778" layer="96" ratio="10" rot="SR270" align="top-left"/>
-<attribute name="NAME" x="-121.6914" y="210.82" size="1.778" layer="95" ratio="10" rot="SR270"/>
-<attribute name="TOLERANCE" x="-129.7686" y="210.82" size="1.778" layer="97" ratio="10" rot="SR270" align="top-left"/>
+<instance part="R206" gate="G$1" x="281.94" y="292.1" smashed="yes" rot="R270">
+<attribute name="VALUE" x="279.1714" y="292.1" size="1.778" layer="96" ratio="10" rot="SR270" align="top-left"/>
+<attribute name="NAME" x="284.7086" y="292.1" size="1.778" layer="95" ratio="10" rot="SR270"/>
+<attribute name="TOLERANCE" x="276.6314" y="292.1" size="1.778" layer="97" ratio="10" rot="SR270" align="top-left"/>
+</instance>
+<instance part="3V3116" gate="G$1" x="281.94" y="297.18" smashed="yes">
+<attribute name="VALUE" x="279.4" y="294.64" size="1.778" layer="96" rot="R90"/>
+</instance>
+<instance part="R203" gate="G$1" x="269.24" y="292.1" smashed="yes" rot="R270">
+<attribute name="VALUE" x="266.4714" y="292.1" size="1.778" layer="96" ratio="10" rot="SR270" align="top-left"/>
+<attribute name="NAME" x="272.0086" y="292.1" size="1.778" layer="95" ratio="10" rot="SR270"/>
+<attribute name="TOLERANCE" x="263.9314" y="292.1" size="1.778" layer="97" ratio="10" rot="SR270" align="top-left"/>
+</instance>
+<instance part="3V3115" gate="G$1" x="269.24" y="297.18" smashed="yes">
+<attribute name="VALUE" x="266.7" y="294.64" size="1.778" layer="96" rot="R90"/>
+</instance>
+<instance part="R202" gate="G$1" x="246.38" y="292.1" smashed="yes" rot="R270">
+<attribute name="VALUE" x="243.6114" y="292.1" size="1.778" layer="96" ratio="10" rot="SR270" align="top-left"/>
+<attribute name="NAME" x="249.1486" y="292.1" size="1.778" layer="95" ratio="10" rot="SR270"/>
+<attribute name="TOLERANCE" x="241.0714" y="292.1" size="1.778" layer="97" ratio="10" rot="SR270" align="top-left"/>
+</instance>
+<instance part="3V3113" gate="G$1" x="246.38" y="297.18" smashed="yes">
+<attribute name="VALUE" x="243.84" y="294.64" size="1.778" layer="96" rot="R90"/>
+</instance>
+<instance part="R201" gate="G$1" x="233.68" y="292.1" smashed="yes" rot="R270">
+<attribute name="VALUE" x="230.9114" y="292.1" size="1.778" layer="96" ratio="10" rot="SR270" align="top-left"/>
+<attribute name="NAME" x="236.4486" y="292.1" size="1.778" layer="95" ratio="10" rot="SR270"/>
+<attribute name="TOLERANCE" x="228.3714" y="292.1" size="1.778" layer="97" ratio="10" rot="SR270" align="top-left"/>
 </instance>
-<instance part="3V3112" gate="G$1" x="-124.46" y="215.9" smashed="yes">
-<attribute name="VALUE" x="-127" y="213.36" size="1.778" layer="96" rot="R90"/>
+<instance part="3V3112" gate="G$1" x="233.68" y="297.18" smashed="yes">
+<attribute name="VALUE" x="231.14" y="294.64" size="1.778" layer="96" rot="R90"/>
 </instance>
 <instance part="D201" gate="R" x="-88.9" y="60.96" smashed="yes">
@@
 <pinref part="R206" gate="G$1" pin="2"/>
 <pinref part="3V3116" gate="G$1" pin="3V3"/>
-<wire x1="-76.2" y1="210.82" x2="-76.2" y2="215.9" width="0.1524" layer="91"/>
+<wire x1="281.94" y1="292.1" x2="281.94" y2="297.18" width="0.1524" layer="91"/>
 </segment>
 <segment>
 <pinref part="R203" gate="G$1" pin="2"/>
 <pinref part="3V3115" gate="G$1" pin="3V3"/>
-<wire x1="-88.9" y1="210.82" x2="-88.9" y2="215.9" width="0.1524" layer="91"/>
+<wire x1="269.24" y1="292.1" x2="269.24" y2="297.18" width="0.1524" layer="91"/>
 </segment>
 <segment>
 <pinref part="R202" gate="G$1" pin="2"/>
 <pinref part="3V3113" gate="G$1" pin="3V3"/>
-<wire x1="-111.76" y1="210.82" x2="-111.76" y2="215.9" width="0.1524" layer="91"/>
+<wire x1="246.38" y1="292.1" x2="246.38" y2="297.18" width="0.1524" layer="91"/>
 </segment>
 <segment>
 <pinref part="R201" gate="G$1" pin="2"/>
 <pinref part="3V3112" gate="G$1" pin="3V3"/>
-<wire x1="-124.46" y1="210.82" x2="-124.46" y2="215.9" width="0.1524" layer="91"/>
+<wire x1="233.68" y1="292.1" x2="233.68" y2="297.18" width="0.1524" layer="91"/>
 </segment>
 <segment>
@@
 <net name="SYS_I2C_SDA" class="0">
 <segment>
-<label x="-124.46" y="193.04" size="1.778" layer="95" rot="R270" xref="yes"/>
-<wire x1="-124.46" y1="198.12" x2="-124.46" y2="193.04" width="0.1524" layer="91"/>
+<label x="233.68" y="274.32" size="1.778" layer="95" rot="R270" xref="yes"/>
+<wire x1="233.68" y1="279.4" x2="233.68" y2="274.32" width="0.1524" layer="91"/>
 <pinref part="R201" gate="G$1" pin="1"/>
 </segment>
@@
 <net name="SYS_I2C_SCL" class="0">
 <segment>
-<label x="-111.76" y="193.04" size="1.778" layer="95" rot="R270" xref="yes"/>
-<wire x1="-111.76" y1="198.12" x2="-111.76" y2="193.04" width="0.1524" layer="91"/>
+<label x="246.38" y="274.32" size="1.778" layer="95" rot="R270" xref="yes"/>
+<wire x1="246.38" y1="279.4" x2="246.38" y2="274.32" width="0.1524" layer="91"/>
 <pinref part="R202" gate="G$1" pin="1"/>
 </segment>
@@
 </segment>
 <segment>
-<wire x1="-88.9" y1="198.12" x2="-88.9" y2="193.04" width="0.1524" layer="91"/>
-<label x="-88.9" y="193.04" size="1.778" layer="95" rot="R270" xref="yes"/>
+<wire x1="269.24" y1="279.4" x2="269.24" y2="274.32" width="0.1524" layer="91"/>
+<label x="269.24" y="274.32" size="1.778" layer="95" rot="R270" xref="yes"/>
 <pinref part="R203" gate="G$1" pin="1"/>
 </segment>
@@
 </segment>
 <segment>
-<wire x1="-76.2" y1="198.12" x2="-76.2" y2="193.04" width="0.1524" layer="91"/>
-<label x="-76.2" y="193.04" size="1.778" layer="95" rot="R270" xref="yes"/>
+<wire x1="281.94" y1="279.4" x2="281.94" y2="274.32" width="0.1524" layer="91"/>
+<label x="281.94" y="274.32" size="1.778" layer="95" rot="R270" xref="yes"/>
 <pinref part="R206" gate="G$1" pin="1"/>
 </segment>
@@
 <text x="124.46" y="30.48" size="1.778" layer="97" align="center">3.3V</text>
 <text x="124.46" y="38.1" size="1.778" layer="97" align="center">2.5V</text>
-<text x="170.18" y="45.72" size="1.778" layer="97" align="center">0.625V</text>
+<text x="170.18" y="45.72" size="1.778" layer="97" align="center">0.675V</text>
 <wire x1="38.1" y1="43.18" x2="48.26" y2="43.18" width="0.1524" layer="97"/>
 <wire x1="38.1" y1="48.26" x2="38.1" y2="43.18" width="0.1524" layer="97"/>

Commit message: PCB routing
Signed-off-by: João Silva <jgc3silva@gmail.com>
Parts:
- removed C1258: 4.7uF, Capacitor:CAPACITOR-0603
- removed C1259: 10uF, Capacitor:CAPACITOR-0402
- removed C3: 1uF, Capacitor:CAPACITOR-0402
- removed C4, C710: 100nF, Capacitor:CAPACITOR-0402
- removed C428: 10pF, Capacitor:CAPACITOR-0402
- removed D1: SMAJ20A, TVS:SMAJ20A
- removed FB701: 1uH, Inductor:FERRITE-0603
- removed R1: 22 Ohms, Resistor:RESISTOR-0402
- removed R11, R12: 2.2K Ohms, Resistor:RESISTOR-0402
- removed R1129: 51.1K Ohms, Resistor:RESISTOR-0402
- removed R1130: 0 Ohms, Resistor:RESISTOR-0402
- removed R1216: 294K Ohms, Resistor:RESISTOR-0402
- removed R13: 49.9 Ohms, Resistor:RESISTOR-0402
- removed R329, R330: 40.2 Ohms, Resistor:RESISTOR-0402
- removed R7: 4.7K Ohms, Resistor:RESISTOR-0402
- removed R8: 1K Ohms, Resistor:RESISTOR-0402
- removed RFCON401: RFCON-U.FL, RF Connector:RFCON-U.FL
- removed TP11: TESTPOINT-0.7MM, PADs:TESTPOINT-0.7MM
- removed U2: ADP7142AUJZ-1.8, Analog Devices:ADP7142AUJZ-1.8
- removed U303: DSC1203DA3-333M3333, Microchip:DSC1203DA3-333M3333
- removed U402: LTC6957-3, Analog Devices:LTC6957-3
- removed U403: TG2520SMN-40.0000M, Crystal:TG2520SMN-40.0000M
- removed U903: SI5351C-B-GM, Silicon Labs:SI5351C-B-GM
- added C105: 10uF, Capacitor:CAPACITOR-0402
- added C106, C108: 1uF, Capacitor:CAPACITOR-0402
- added C107, C272, C624: 100nF, Capacitor:CAPACITOR-0402
- added CON102: FPC-22P, Generic Connector:FPC-22P
- added D1002: SMAJ20A, TVS:SMAJ20A
- added D1004: B0530W, Generic Diode:B0530W
- added D505, D506, D507, D508: LED0603, LED:LED0603
- added D509, D510, D511, D512, D601, D602: PGB1010402, TVS:PGB1010402
- added R1013, R1122, R217, R218: 10K Ohms, Resistor:RESISTOR-0402
- added R1123: DNP, Resistor:RESISTOR-0402
- added R115, R116: 2.2K Ohms, Resistor:RESISTOR-0402
- added R301: 240 Ohms, Resistor:RESISTOR-0402
- added R326: 40.2 Ohms, Resistor:RESISTOR-0402
- added R615: 49.9 Ohms, Resistor:RESISTOR-0402
- added R913: 0 Ohms, Resistor:RESISTOR-0402
- added RFCON101: RFCON-SMA-EDGE, RF Connector:RFCON-SMA-EDGE
- added U301: MT41K256M16TW-125, Micron:MT41K256M16TW-125
- C1, C421, C620: value 100nF -> 10nF
- C102: device Capacitor:CAPACITOR-0402 -> Capacitor:CAPACITOR-0603
- C103: value 100nF -> 10uF; device Capacitor:CAPACITOR-0402 -> Capacitor:CAPACITOR-0603
- C104: value 1uF -> 10uF; device Capacitor:CAPACITOR-0402 -> Capacitor:CAPACITOR-0603
- C1249: value 100nF -> 470pF
- C1251: value 470pF -> 100nF
- C1252: value 100nF -> 100uF; device Capacitor:CAPACITOR-0402 -> Capacitor:CAPACITOR-1206
- C1253: value 100uF -> 10uF; device Capacitor:CAPACITOR-1206 -> Capacitor:CAPACITOR-0402
- C1254, C1255: value 10uF -> 100nF
- C1256: value 100nF -> 4.7uF; device Capacitor:CAPACITOR-0402 -> Capacitor:CAPACITOR-0603
- C1257: value 100nF -> 10uF
- C2, C408, C409, C413, C414, C420: value 1uF -> 10nF
- C403: value 1uF -> DNP
- C405, C426, C902: value 100nF -> 1uF
- C406: value 10nF -> 10pF
- C407: value 10nF -> 100nF
- C410: value 10uF -> 1uF
- C411, C416, C417: value 10nF -> 1uF
- C412: value 10nF -> 10uF
- C423, C542, C543: value 1nF -> 100nF
- C427: value DNP -> 1nF
- C536, C537, C548, C549, C550: value 18pF -> 1nF
- C538, C539, C544, C545, C546: value 1nF -> 18pF
- C540, C541: value 100nF -> 1nF
- C605, C608, C611: value 22uF -> 100nF
- C606, C609, C614: value 100nF -> 22uF
- C615: value 47nF -> 100nF
- C616: value 2.7nF -> 47nF
- C617: value 680pF -> 2.7nF
- C618: value 10nF -> 680pF
- C905, C906: value 100nF -> 10pF
- C907, C908: value 10pF -> 100nF
- CON1: value FPC-22P -> 4P-SH-TOP; device Generic Connector:FPC-22P -> JST:4P-SH-TOP
- D1001: value B0530W -> PGB102ST23; device Generic Diode:B0530W -> TVS:PGB102ST23
- D501, D502, D503, D504: value LED0603 -> PGB1010402; device LED:LED0603 -> TVS:PGB1010402; COLOR YELLOW -> (none)
- Q1101: value AO4805 -> AO3400; device Alpha Omega:AO4805 -> Alpha Omega:AO3400
- Q1102: value AO3400 -> AO4805; device Alpha Omega:AO3400 -> Alpha Omega:AO4805
- R101: value 2.2K Ohms -> 1K Ohms
- R1010, R1119: value 10K Ohms -> 1K Ohms
- R102: value 10K Ohms -> 2.2K Ohms
- R103: value TBD Ohms -> 10K Ohms
- R104: value 0 Ohms -> TBD Ohms
- R106: value DNP -> 1K Ohms
- R107: value 1K Ohms -> 0 Ohms
- R108: value 0 Ohms -> DNP
- R109: value DNP -> 0 Ohms
- R110: value 1K Ohms -> DNP
- R1120, R901: value 10K Ohms -> DNP
- R1121, R603: value 1K Ohms -> 10K Ohms
- R1124, R403: value DNP -> 10K Ohms
- R1125: value DNP -> 36.5K Ohms
- R1126: value 10K Ohms -> 124K Ohms
- R1127: value 36.5K Ohms -> 51.1K Ohms
- R1128: value 124K Ohms -> 0 Ohms
- R1212: value 10K Ohms -> 309K Ohms
- R1213: value 309K Ohms -> 71.5K Ohms
- R1214: value 71.5K Ohms -> 274K Ohms
- R1215: value 274K Ohms -> 294K Ohms
- R201: value 4.7K Ohms -> 22 Ohms
- R202, R203: value 4.7K Ohms -> 330 Ohms
- R205, R207: value 330 Ohms -> 4.7K Ohms
- R208: value 100 Ohms -> 4.7K Ohms; TOLERANCE 1% -> (none)
- R209: value 10K Ohms -> 100 Ohms; TOLERANCE (none) -> 1%
- R210: value 10K Ohms -> 4.7K Ohms
- R304: value 240 Ohms -> 40.2 Ohms
- R401: value 10K Ohms -> 25 Ohms
- R402: value 14.3K Ohms -> 25 Ohms
- R404: value DNP -> 14.3K Ohms
- R602: value 10K Ohms -> 49.9 Ohms
- R607: value 360 Ohms -> 1K Ohms
- R608: value 1K Ohms -> 360 Ohms
- R609: value 49.9 Ohms -> 1K Ohms
- R902: value 10K Ohms -> 0 Ohms
- R905: value 0 Ohms -> 10K Ohms
- U302: value MT41K256M16TW-125 -> DSC1203DA3-333M3333; device Micron:MT41K256M16TW-125 -> Microchip:DSC1203DA3-333M3333
- U901: value 74LVC1G157 -> DSB321SDA; device Logic:74LVC1G157 -> Crystal:DSB321SDA
- U902: value DSB321SDA -> SI5351C-B-GM; device Crystal:DSB321SDA -> Silicon Labs:SI5351C-B-GM
- renumbered D2 to D1003, D3 to D203, D4 to D202, FB1 to FB901, R10 to R216, R2 to R212, R3 to R214, R4 to R215, R5 to R213, R6 to R211, R9 to R219, U1 to U202
Connections:
- net EXT_VIN renamed VEXT_UNFUSED
- net N$110 renamed PM_SPI_MOSI
- net N$112 renamed !PM_SPI_CS
- net N$113 renamed PM_SPI_CLK
- net N$114 renamed PM_SPI_MISO
- net N$115 renamed !PM_SPI_IRQ
- net N$58 renamed VBUS_UNFUSED
- removed net 1V8_TRX_REF: C1255.C1, C426.C1, U2.SENSE/ADJ, U2.VOUT, U403.VDD
- removed net 3V3_DMIC: C711.C1, C712.C1, FB701.2, M701.SEL, M701.VCC, M702.VCC
- removed net CLK_MNGR_CLKIN_SEL: R901.2, U901.1.SEL
- removed net N$111: R1007.2, TP11.TP, U1002.PA07/SPI_MOSI_SI
- removed net N$12: RFCON901.SIGNAL, U901.1.I1
- removed net N$2: U901.1.Y, U903.CLKIN
- removed net N$29: R403.2, RFCON401.SIGNAL
- removed net N$34: C902.C1, C904.C1, C905.C1, FB901.2, U903.VDDOA, U903.VDDOB, U903.VDDOC, U903.VDDOD
- removed net N$57: L1001.1, USB1001.D-
- removed net N$59: L1001.4, USB1001.D+
- removed net N$6: U1102.1.VSENSEN
- removed net TRX_REF_EN: R1211.2, U2.EN
- new net 3V3_CLK_MNGR: C901.C1, C903.C1, C904.C1, C907.C1, FB901.2, U901.VDD, U902.VDDOA, U902.VDDOB, U902.VDDOC, U902.VDDOD
- new net CLK_MNGR_CLKIN: R902.1, U902.CLKIN
- new net CLK_MNGR_EXT_REF: R901.2, R902.2, RFCON901.SIGNAL
- new net CODEC_EXT_DMIC_DATA: CON1-3.S, U701.DMIC2_3/MP5
- new net PM_SPI_MOSI_SI: R1007.2, U1002.PA07/SPI_MOSI_SI
- new net TRX_XTALN: C406.C2, U401.INTERFACE.XTALN
- new net USB_D_UNFILT_N: D1001.C1, L1001.1, USB1001.D-
- new net USB_D_UNFILT_P: D1001.C2, L1001.4, USB1001.D+
- net !CLK_MNGR_IRQ: now also R905.1, U902.!INTR; no longer R904.1, U903.!INTR
- net !CLK_MNGR_OE: now also R904.1, U902.!OE; no longer R902.1, U903.!OE
- net !DDR3_CAS: now also R327.1, U301.!CAS; no longer R329.1, U302.!CAS
- net !DDR3_RAS: now also R324.1, U301.!RAS; no longer R325.1, U302.!RAS
- net !DDR3_RESET: now also U301.!RESET; no longer U302.!RESET
- net !DDR3_WE: now also R323.1, U301.!WE; no longer R324.1, U302.!WE
- net !FPGA_PROGRAM: now also R210.1; no longer R7.1
- net !PMC_RESET: now also R1013.1; no longer R1012.1
- net !TRX_RESET: now also R403.2; no longer R401.2
- net !VBUS_SRC_FAULT: now also R1011.1, U1002.GPIO3; no longer R1010.1
- net 0V675_DDR3_VREF: now also U301.VREFCA, U301.VREFDQ; no longer U302.VREFCA, U302.VREFDQ
- net 0V675_DDR3_VTT: now also R304.1, R313.1, R321.2, R326.2; no longer R312.1, R320.1, R329.2, R330.2
- net 12V0_VSENSE: now also U1002.PA04
- net 1V0_PGOOD: now also R1122.1; no longer R1120.1
- net 1V1_TRX_RX_VCO: now also C426.C1, C427.C1; no longer C424.C1, C425.C1
- net 1V1_TRX_TX_VCO: now also C424.C1, C425.C1; no longer C422.C1, C423.C1
- net 1V2: now also C1255.C1, R1214.2, R209.2; no longer C1259.C1, R1215.2, R208.2
- net 1V2_FB: now also R1214.1, R1215.2; no longer R1215.1, R1216.2
- net 1V2_SS: now also C1249.C1; no longer C1250.C1
- net 1V35: now also U301.VDD, U301.VDDQ; no longer U302.VDD, U302.VDDQ
- net 1V3_TRX: now also C404.C1, C410.C1, C413.C1, C416.C1, C419.C1, C536.C1, C537.C1, C540.C1, C541.C1; no longer C403.C1, C406.C1, C411.C1, C414.C1, C417.C1, C538.C1, C539.C1, C542.C1, C543.C1
- net 1V3_TRX_LO_SYNTH: now also C405.C1, C411.C1, C414.C1, C417.C1, C420.C1; no longer C404.C1, C407.C1, C412.C1, C415.C1, C418.C1
- net 2V5: now also C407.C1; no longer C1249.C1, C405.C1, U2.VIN
- net 2V5_TRX_INTERFACE: now also C412.C1, C415.C1, C418.C1; no longer C410.C1, C413.C1, C416.C1
- net 3V3: now also C1251.C1, C272.C1, C423.C1, C902.C1, C908.C1, R1211.2, R205.2, R207.2, R208.2, R217.2, R218.2, R905.2, U302.!STDBY, U302.VDD; no longer C1.C1, C1253.C1, C3.C1, C421.C1, C710.C1, C901.C1, C903.C1, C906.C1, FB701.1, R1213.2, R201.2, R202.2, R203.2, R209.2, R7.2, R902.2, U303.!STDBY, U303.VDD, U901.PWR.VCC, U903.VDD
- net 3V3_CM4: now also C106.C1, C108.C1, CON102-1.S, R101.2, R103.2, R106.2, R115.2, R116.2; no longer C104.C1, C2.C1, CON1-1.S, R102.2, R107.2, R11.2, R110.2, R12.2
- net 3V3_CM4_SD: now also C105.C1; no longer C102.C1
- net 3V3_CODEC: now also C1253.C1, C711.C1, C712.C1, CON1-1.S, M701.SEL, M701.VCC, M702.VCC; no longer C1254.C1
- net 3V3_FB: now also R1212.1, R1213.2; no longer R1213.1, R1214.2
- net 3V3_PGOOD: now also R1211.1; no longer R1212.1
- net 3V3_PM: now also R1011.2, R1013.2; no longer R1010.2, R1012.2
- net 3V3_SS: now also C1250.C1; no longer C1251.C1
- net 3V3_SYNTH_IN_PD_FB: now also C604.C1, C607.C1, C610.C1, R604.2, R606.2; no longer C603.C1, C606.C1, C609.C1, R603.2, R605.2
- net 3V3_SYNTH_VCO_RF: now also C605.C1, C608.C1, C611.C1; no longer C604.C1, C607.C1, C610.C1
- net 3V3_TRX_GPO: now also C421.C1, C422.C1; no longer C419.C1, C420.C1
- net 3V5_VIN_REG_DRVCC: now also R1120.2, R1123.2; no longer R1125.2, R1126.2
- net 5V0: now also C102.C1, C103.C1, C104.C1, C1254.C1, R1122.2; no longer C1258.C1, R1120.2
- net 5V0_PGOOD: now also R1121.1; no longer R1119.1
- net 5V0_TRX_BIAS_T1: now also D505.A; no longer D501.A
- net 5V0_TRX_BIAS_T2: now also D506.A; no longer D502.A
- net 5V0_TRX_PA1: now also C542.C1, C548.C1, C551.C1, D507.A; no longer C540.C1, C544.C1, C547.C1, D503.A
- net 5V0_TRX_PA2: now also C543.C1, C549.C1, C552.C1, D508.A; no longer C541.C1, C545.C1, C548.C1, D504.A
- net AUDIO_I2C_SCL: now also R208.1; no longer R206.1
- net AUDIO_I2C_SDA: now also R207.1; no longer R203.1
- net CLK_MNGR_CLK0: now also R906.2, U902.CLK0; no longer R905.2, U903.CLK0
- net CLK_MNGR_CLK1: now also R910.2, U902.CLK1; no longer R909.2, U903.CLK1
- net CLK_MNGR_CLK2: now also R907.2, U902.CLK2; no longer R906.2, U903.CLK2
- net CLK_MNGR_CLK3: now also R911.2, U902.CLK3; no longer R910.2, U903.CLK3
- net CLK_MNGR_CLK4: now also R908.2, U902.CLK4; no longer R907.2, U903.CLK4
- net CLK_MNGR_CLK5: now also R912.2, U902.CLK5; no longer R911.2, U903.CLK5
- net CLK_MNGR_CLK6: now also R909.2, U902.CLK6; no longer R908.2, U903.CLK6
- net CLK_MNGR_CLK7: now also R913.2, U902.CLK7; no longer R912.2, U903.CLK7
- net CLK_MNGR_REF_ACC: now also C906.C2, U902.XA; no longer C908.C2, U903.XA
- net CLK_MNGR_REF_DCC: now also C905.C1, C906.C1, U901.CLK; no longer C907.C1, C908.C1, U902.CLK
- net CM4_CAM0_CSI_C_N: now also CON101-15.S; no longer CON1-15.S
- net CM4_CAM0_CSI_C_P: now also CON101-14.S; no longer CON1-14.S
- net CM4_CAM0_CSI_D0_N: now also CON101-21.S; no longer CON1-21.S
- net CM4_CAM0_CSI_D0_P: now also CON101-20.S; no longer CON1-20.S
- net CM4_CAM0_CSI_D1_N: now also CON101-18.S; no longer CON1-18.S
- net CM4_CAM0_CSI_D1_P: now also CON101-17.S; no longer CON1-17.S
- net CM4_CAM0_SCL: now also CON101-3.S, R114.1; no longer CON1-3.S, R12.1
- net CM4_CAM0_SDA: now also CON101-2.S, R113.1; no longer CON1-2.S, R11.1
- net CM4_CAM1_CSI_C_N: now also CON102-15.S; no longer CON101-15.S
- net CM4_CAM1_CSI_C_P: now also CON102-14.S; no longer CON101-14.S
- net CM4_CAM1_CSI_D0_N: now also CON102-21.S; no longer CON101-21.S
- net CM4_CAM1_CSI_D0_P: now also CON102-20.S; no longer CON101-20.S
- net CM4_CAM1_CSI_D1_N: now also CON102-18.S; no longer CON101-18.S
- net CM4_CAM1_CSI_D1_P: now also CON102-17.S; no longer CON101-17.S
- net CM4_CAM1_CSI_D2_N: now also CON102-12.S; no longer CON101-12.S
- net CM4_CAM1_CSI_D2_P: now also CON102-11.S; no longer CON101-11.S
- net CM4_CAM1_CSI_D3_N: now also CON102-9.S; no longer CON101-9.S
- net CM4_CAM1_CSI_D3_P: now also CON102-8.S; no longer CON101-8.S
- net CM4_CAM1_SCL: now also CON102-3.S, R116.1; no longer CON101-3.S, R114.1
- net CM4_CAM1_SDA: now also CON102-2.S, R115.1; no longer CON101-2.S, R113.1
- net CM4_CAM_GPIO: now also CON102-6.S; no longer CON1-6.S
- net CM4_GLOBAL_EN: now also R102.2; no longer R101.2
- net CM4_PTP_PPS: now also R110.2; no longer R108.2
- net CM4_SD_PWR_EN: now also R103.1; no longer R102.1
- net CODEC_DMIC_CLK: now also CON1-2.S
- net DDR3_A0: now also R304.2, U301.A0; no longer R305.2, U302.A0
- net DDR3_A1: now also R313.2, U301.A1; no longer R314.2, U302.A1
- net DDR3_A10: now also R309.2, U301.A10/AP; no longer R310.2, U302.A10/AP
- net DDR3_A11: now also R318.2, U301.A11; no longer R319.2, U302.A11
- net DDR3_A12: now also R310.2, U301.A12/!BC; no longer R311.2, U302.A12/!BC
- net DDR3_A13: now also R319.2, U301.A13; no longer R320.2, U302.A13
- net DDR3_A14: now also R311.2, U301.A14; no longer R312.2, U302.A14
- net DDR3_A2: now also R305.2, U301.A2; no longer R306.2, U302.A2
- net DDR3_A3: now also R314.2, U301.A3; no longer R315.2, U302.A3
- net DDR3_A4: now also R306.2, U301.A4; no longer R307.2, U302.A4
- net DDR3_A5: now also R315.2, U301.A5; no longer R316.2, U302.A5
- net DDR3_A6: now also R307.2, U301.A6; no longer R308.2, U302.A6
- net DDR3_A7: now also R316.2, U301.A7; no longer R317.2, U302.A7
- net DDR3_A8: now also R308.2, U301.A8; no longer R309.2, U302.A8
- net DDR3_A9: now also R317.2, U301.A9; no longer R318.2, U302.A9
- net DDR3_BA0: now also R322.1, U301.BA0; no longer R323.1, U302.BA0
- net DDR3_BA1: now also R325.1, U301.BA1; no longer R327.1, U302.BA1
- net DDR3_BA2: now also R321.1, U301.BA2; no longer R322.1, U302.BA2
- net DDR3_CLK_EN: now also R328.1, U301.CKE; no longer R330.1, U302.CKE
- net DDR3_CLK_IN_N: now also U302.!CLK; no longer U303.!CLK
- net DDR3_CLK_IN_P: now also U302.CLK; no longer U303.CLK
- net DDR3_CLK_N: now also R320.1, U301.!CK; no longer R321.1, U302.!CK
- net DDR3_CLK_P: now also R312.2, U301.CK; no longer R313.2, U302.CK
- net DDR3_DM0: now also U301.LDM; no longer U302.LDM
- net DDR3_DM1: now also U301.UDM; no longer U302.UDM
- net DDR3_DQ0: now also U301.DQ0; no longer U302.DQ0
- net DDR3_DQ1: now also U301.DQ1; no longer U302.DQ1
- net DDR3_DQ10: now also U301.DQ10; no longer U302.DQ10
- net DDR3_DQ11: now also U301.DQ11; no longer U302.DQ11
- net DDR3_DQ12: now also U301.DQ12; no longer U302.DQ12
- net DDR3_DQ13: now also U301.DQ13; no longer U302.DQ13
- net DDR3_DQ14: now also U301.DQ14; no longer U302.DQ14
- net DDR3_DQ15: now also U301.DQ15; no longer U302.DQ15
- net DDR3_DQ2: now also U301.DQ2; no longer U302.DQ2
- net DDR3_DQ3: now also U301.DQ3; no longer U302.DQ3
- net DDR3_DQ4: now also U301.DQ4; no longer U302.DQ4
- net DDR3_DQ5: now also U301.DQ5; no longer U302.DQ5
- net DDR3_DQ6: now also U301.DQ6; no longer U302.DQ6
- net DDR3_DQ7: now also U301.DQ7; no longer U302.DQ7
- net DDR3_DQ8: now also U301.DQ8; no longer U302.DQ8
- net DDR3_DQ9: now also U301.DQ9; no longer U302.DQ9
- net DDR3_DQS0_N: now also U301.!LDQS; no longer U302.!LDQS
- net DDR3_DQS0_P: now also U301.LDQS; no longer U302.LDQS
- net DDR3_DQS1_N: now also U301.!UDQS; no longer U302.!UDQS
- net DDR3_DQS1_P: now also U301.UDQS; no longer U302.UDQS
- net DDR3_ODT: now also R326.1, U301.ODT; no longer R328.1, U302.ODT
- net EXT_CLK_OUT: now also R913.1; no longer R912.1
- net FPGA_CLK0: now also R906.1; no longer R905.1
- net FPGA_CLK1: now also R910.1; no longer R909.1
- net FPGA_CLK2: now also R907.1; no longer R906.1
- net FPGA_CLK3: now also R911.1; no longer R910.1
- net FPGA_TDI: now also R217.1; no longer R209.1
- net FPGA_TMS: now also R218.1; no longer R210.1
- net GND: now also C105.C2, C106.C2, C107.C2, C108.C2, C272.C2, C536.C2, C537.C2, C549.C2, C551.C2, C552.C2, C620.C2, C908.C2, CON102-10.S, CON102-13.S, CON102-16.S, CON102-19.S, CON102-22.S, CON102-4.S, CON102-7.S, D1001.A, D1002.A, D501.2, D502.2, D503.2, D504.2, D509.2, D510.2, D511.2, D512.2, D601.2, D602.2, Q1101.S, R1012.1, R102.1, R107.1, R108.1, R1125.1, R1126.1, R1213.1, R1215.1, R301.1, R403.1, R603.1, R605.1, R607.1, R615.1, U1102.1.VSENSEN, U201.BANK216-GTP.MGTPRXN1, U201.BANK216-GTP.MGTPRXP1, U301.!CS, U301.VSS, U301.VSSQ, U302.GND, U901.GND; no longer C1258.C2, C1259.C2, C3.C2, C4.C2, C406.C2, C538.C2, C539.C2, C544.C2, C545.C2, C547.C2, C710.C2, C906.C2, CON1-10.S, CON1-13.S, CON1-16.S, CON1-19.S, CON1-22.S, CON1-7.S, D1.A, Q1102.S, R101.1, R1011.1, R103.1, R106.1, R1129.1, R1130.1, R1211.1, R1214.1, R1216.1, R13.1, R304.1, R401.1, R604.1, R606.1, R613.1, RFCON401.GND, U2.GND, U302.!CS, U302.VSS, U302.VSSQ, U303.GND, U403.GND, U901.PWR.GND, U903.GND
- net N$101: now also C616.C1, R608.1; no longer C615.C1, R607.1
- net N$116: now also R109.1; no longer R108.1
- net N$117: now also R110.1; no longer R109.1
- net N$118: now also R107.2; no longer R105.2
- net N$119: now also R105.2; no longer R104.2
- net N$120: now also R108.2; no longer R106.2
- net N$121: now also R101.1; no longer R107.1
- net N$123: now also R106.1; no longer R110.1
- net N$148: now also R1119.1; no longer R1121.1
- net N$16: now also C550.C1; no longer C546.C1
- net N$18: now also C545.C2; no longer C550.C2
- net N$19: now also R1010.1; no longer R8.1
- net N$20: now also C544.C2; no longer C549.C2
- net N$21: now also Q1102.1.G, Q1102.2.G; no longer Q1101.1.G, Q1101.2.G
- net N$22: now also C547.C2; no longer C552.C2
- net N$23: now also C546.C2; no longer C551.C2
- net N$31: now also R209.1; no longer R208.1
- net N$36: now also Q1101.D; no longer Q1102.D
- net N$4: now also Q1102.1.S, Q1102.2.S; no longer Q1101.1.S, Q1101.2.S
- net N$40: now also C107.C1; no longer C103.C1
- net N$70: now also D507.C; no longer D503.C
- net N$73: now also R301.2, U301.ZQ; no longer R304.2, U302.ZQ
- net N$74: now also R104.2; no longer R103.2
- net N$79: now also D508.C; no longer D504.C
- net N$8: now also R404.2; no longer R402.2
- net N$81: now also D505.C; no longer D501.C
- net N$83: now also D506.C; no longer D502.C
- net N$87: now also R312.1, R320.2; no longer R313.1, R321.2
- net N$94: now also D1004.A; no longer D1001.A
- net N$98: now also C615.C1; no longer C614.C1
- net PLL_REF_DCC: now also C403.C1, C406.C1, R401.1, R402.2; no longer C427.C1, C428.C1, R403.1, R404.2, U403.CLK
- net PMC_SWO: now also R1012.2; no longer R1011.2
- net SYNTH_CE: now also R603.2; no longer R602.2
- net SYNTH_CPBIAS: now also C614.C1; no longer C613.C1
- net SYNTH_CPOUT: now also C617.C1, R609.2; no longer C616.C1, R607.2
- net SYNTH_REFIN_N: now also C603.C1, R606.1, R607.2; no longer C4.C1, R605.1, R606.2
- net SYNTH_REFIN_P: now also R604.1, R605.2; no longer R603.1, R604.2
- net SYNTH_REF_CLK: now also R602.2; no longer R13.2
- net SYNTH_RFOUTA_ACC_N: now also C621.C2, R614.2; no longer C620.C2, R613.2
- net SYNTH_RFOUTA_ACC_P: now also C623.C2, D601.1; no longer C622.C2
- net SYNTH_RFOUTA_BIAS: now also C1.C1, C619.C1, R610.2, R612.2; no longer C618.C1, R609.2, R611.2
- net SYNTH_RFOUTA_N: now also C621.C1, R612.1; no longer C620.C1, R611.1
- net SYNTH_RFOUTA_P: now also C623.C1, R610.1; no longer C622.C1, R609.1
- net SYNTH_RFOUTB_ACC_N: now also C622.C2, R615.2; no longer C621.C2, R614.2
- net SYNTH_RFOUTB_ACC_P: now also C624.C2, D602.1; no longer C623.C2
- net SYNTH_RFOUTB_BIAS: now also C2.C1, C620.C1, R611.2, R613.2; no longer C619.C1, R610.2, R612.2
- net SYNTH_RFOUTB_N: now also C622.C1, R613.1; no longer C621.C1, R612.1
- net SYNTH_RFOUTB_P: now also C624.C1, R611.1; no longer C623.C1, R610.1
- net SYNTH_VREFVCO1: now also C612.C1; no longer C611.C1
- net SYNTH_VREFVCO2: now also C613.C1; no longer C612.C1
- net SYNTH_VREGVCO1: now also C606.C1; no longer C605.C1
- net SYNTH_VREGVCO2: now also C609.C1; no longer C608.C1
- net SYNTH_VTUNE: now also C618.C1, R609.1; no longer C617.C1, R608.1
- net SYS_I2C_SCL: now also R206.1, U902.SCL; no longer R202.1, U903.SCL
- net SYS_I2C_SDA: now also R205.1, U902.SDA; no longer R201.1, U903.SDA
- net TRX_CLK_OUT: no longer U901.1.I0
- net TRX_REF_CLK: now also R401.2; no longer C428.C2, U401.INTERFACE.XTALN
- net TRX_RX1A: now also D501.1
- net TRX_RX1C_DCC: now also D503.1
- net TRX_RX2A: now also D502.1
- net TRX_RX2C_DCC: now also D504.1
- net TRX_SYNC_IN: now also R201.2; no longer R1.2
- net TRX_TX1A: now also D509.1
- net TRX_TX1A_N: now also C544.C1; no longer C549.C1
- net TRX_TX1A_P: now also C545.C1; no longer C550.C1
- net TRX_TX1B: now also C538.C1; no longer C536.C1
- net TRX_TX1B_AMP_ACC: now also D511.1
- net TRX_TX1B_DCC: now also C538.C2; no longer C536.C2
- net TRX_TX2A: now also D510.1
- net TRX_TX2A_N: now also C546.C1; no longer C551.C1
- net TRX_TX2A_P: now also C547.C1; no longer C552.C1
- net TRX_TX2B: now also C539.C1; no longer C537.C1
- net TRX_TX2B_AMP: now also D512.1
- net TRX_TX2B_DCC: now also C539.C2; no longer C537.C2
- net TRX_TXMON2: now also C550.C2; no longer C546.C2
- net VBUS: now also D1002.C, D1004.C, Q1102.2.D; no longer D1.C, D1001.C, Q1101.2.D
- net VBUS_SNK_EN: now also Q1101.G, U1002.PA27/GPIO9; no longer Q1102.G
- net VBUS_SRC_EN: now also U1002.GPIO2
- net VBUS_VSENSE: now also U1002.PA02
- net VEXT_EN: now also U1002.PA06
- net VEXT_VSENSE: now also U1002.PA05
- net VIN: now also Q1102.1.D; no longer Q1101.1.D
- net VIN_REG_ASEL: now also R1128.2; no longer R1130.2
- net VIN_REG_PWM_CFG: now also R1127.2; no longer R1129.2
- net VIN_REG_RUN0: now also R1123.1; no longer R1125.1
- net VIN_REG_SHARE_CLK: now also R1124.1; no longer R1126.1
- net VIN_REG_VOUT0_CFG: now also R1126.2; no longer R1128.2
- net VIN_REG_VOUT1_CFG: now also R1125.2; no longer R1127.2
- net VIN_REG_WP: now also R1120.1; no longer R1124.1
- net VIN_VSENSE: now also U1002.PA03
Other:
- note added: "Digital Rail FPGA GTP VTT"
- note added: "Load switch drops at most 62.5 mV @ 500 mA Diode drops at most 430 mV @ 500 mA With 5V0 bus regulated to 5.2 V, this should ensure a worst case sourced VBUS of about 4.7 V. Slightly out of spec, but should work. :)"
- note added: "XTALN typical swing is 1.3 Vpp."
- note removed: "ADP150 1.8V @ 150mA"
- note removed: "Analog Rail AD9361 Reference TCXO"
- note removed: "Digital Rail FPGA GTP VTT, USB FIFO Core"
- note removed: "Enable"
- note removed: "TRX_REF_CLK max swing is 1.3 Vpp. If an external reference is applied that does not match this level, R401 and R402 can form a voltage divider"
- note removed: "TVS"
- moved on the sheet: C1005, C1006, C102, C103, C104, C1249, C1250, C1251, C1252, C1253, C1254, C1255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
